File: Power_Supplies/PREAMPS.kicad_sch (KiCad schematic)
At the start: 24 parts, among them J3 XLR3, SW1 SW_Push, U12 SSM2019BRNZ

Commit message: Working on preamp
Parts:
- added C115: 0.1uF, Capacitor_SMD:C_0402_1005Metric, symbol Device:C
- added J5: AudioJack3, symbol Connector_Audio:AudioJack3
- added R51: 1M, Resistor_SMD:R_0805_2012Metric, symbol Device:R
- added RV1: 10k, symbol Device:R_Potentiometer
- added U13: OPA2134, symbol Amplifier_Operational:OPA2134
Connections:
- net AGND: now also J5.S; no longer DZ2.2 (A), DZ4.2 (A)
- net PRE_VIRTUAL_GND: now also DZ2.2 (A), DZ4.2 (A), R51.1
- net PREAMP_STAGE1_OUTPUT renamed PREAMP1_MIC_OUT
- new net: C115.1, R51.2, U13.3 (+)
- new net: C115.2, J5.T
- new net: RV1.1, U13.1, U13.2 (-)
- new net PREAMP1_HIZ_OUT: RV1.2
Other:
- note added: "Mic Preamp Front-end (Phantom Power)"
- note added: "Preamp Hi-Z Stage (Impedance Buffer)"
- note added: "Preamp Mic Stage"
- note removed: "Preamp Front-end (Phantom Power)"
- note removed: "Preamp Stage 1"
- title: (none) -> Preamps
