File: Power_Supplies/XCORE.kicad_sch (KiCad schematic)
At the start: 7 parts, among them U10 XU316-1024-TQ128-I24, U11 W25Q64JVSSIQ (FLASH MEMORY), X1 FA-238 24.0000MB-C0 (CRYSTAL)

Commit message: Add files via upload
Parts:
- C100, C101: value 18pf -> 18pF; footprint (none) -> Capacitor_SMD:C_0402_1005Metric
- R28, R29: footprint (none) -> Resistor_SMD:R_0805_2012Metric
Changed lines of the file:
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@@
 	(generator "eeschema")
 	(generator_version "8.0")
-	(paper "A2")
+	(paper "A4")
 	(title_block
 		(title "XCORE")
@@
 			)
 		)
-		(property "Footprint" ""
+		(property "Footprint" "Resistor_SMD:R_0805_2012Metric"
 			(at 102.87 25.908 90)
 			(effects
@@
 			)
 		)
-		(property "Value" "18pf"
+		(property "Value" "18pF"
 			(at 132.08 138.4299 0)
 			(effects
@@
 			)
 		)
-		(property "Footprint" ""
+		(property "Footprint" "Capacitor_SMD:C_0402_1005Metric"
 			(at 129.2352 140.97 0)
 			(effects
@@
 			)
 		)
-		(property "Footprint" ""
+		(property "Footprint" "Resistor_SMD:R_0805_2012Metric"
 			(at 123.952 146.05 90)
 			(effects
@@
 			)
 		)
-		(property "Value" "18pf"
+		(property "Value" "18pF"
 			(at 168.91 156.2099 0)
 			(effects
@@
 			)
 		)
-		(property "Footprint" ""
+		(property "Footprint" "Capacitor_SMD:C_0402_1005Metric"
 			(at 166.0652 158.75 0)
 			(effects

Commit message: Finished HiZ Inputs
Other:
- moved on the sheet: C100, C101, R28, R29, U10A, U10B, U11, X1
