File: Power_Supplies/_autosave-XCORE.kicad_sch (KiCad schematic)
At the start: 11 parts, among them J22 FTSH-110-01-F-DV-K XTAG HEADER, U10 XU316-1024-TQ128-I24, U11 W25Q64JVSSIQ (FLASH MEMORY), X1 FA-238 24.0000MB-C0 (CRYSTAL)

Commit message: Working on MCU IO
Connections:
- net 0.9V: now also U10.11 (VDD), U10.18 (VDD), U10.39 (VDD), U10.50 (VDD), U10.54 (VDD), U10.68 (VDD), U10.85 (VDD), U10.95 (VDD)
- net AGND: now also U10.30 (GND)
- no-connect marks 0 -> 8
