File: Power_Supplies/ADC.kicad_sch (KiCad schematic)
At the start: 61 parts, among them IC1 PCM4201PWR, IC5 PCM1808PWRG4, J3 031-5640-1010, J5 AudioJack2, U14 MCP6001T-E/OT, U15 MCP6001T-E/OT, U16 OPA2134, U17 LM27761

Commit message: Add files via upload
Parts:
- removed C42, C47, C49: 150p, Capacitor_SMD:C_0402_1005Metric, symbol Device:C
- removed C43, C44, C48: 100n, Capacitor_SMD:C_0402_1005Metric, symbol Device:C
- removed C45, C46: 1n, Capacitor_SMD:C_0402_1005Metric, symbol Device:C
- removed C50, C70, C72, C73: 10uF, Capacitor_SMD:CP_Elec_4x5.8, symbol Device:C_Polarized_US
- removed C51, C68: 0.1uF, Capacitor_SMD:C_0805_2012Metric, symbol Device:C
- removed C74: 1uF, Capacitor_SMD:CP_Elec_4x5.8, symbol Device:C_Polarized_US
- removed D3: PESD3V3L1BA,115, Diode_SMD:D_SOD-323, symbol Device:D_TVS
- removed IC5: PCM1808PWRG4, SamacSys_Parts:SOP65P640X120-14N, symbol SamacSys_Parts:PCM1808PWRG4
- removed J3: 031-5640-1010, PhilsLab_Footprints_KiCad6:AMPHENOL-BNC-031-5640-1010, symbol Connector:Conn_Coaxial
- removed U14, U15: MCP6001T-E/OT, Package_TO_SOT_SMD:SOT-23-5, symbol Amplifier_Operational:MCP6001-OT
- added C121, C122, C123, C124, C70, C77, C84: 1nF, Capacitor_SMD:C_0402_1005Metric, symbol Device:C
- added C125, C127, C128, C130, C131, C133, C134, C136, C73, C78, C80, C85, C87: 100pF, Capacitor_SMD:C_0805_2012Metric, symbol Device:C
- added C126, C129, C132, C135, C72, C79, C86: 0.022uF, Capacitor_SMD:C_0805_2012Metric, symbol Device:C
- added C50, C67, C74, C81, C88, C89, C90, C91: 100uF, Capacitor_SMD:C_0805_2012Metric, symbol Device:C
- added C51, C68, C82, C92, C93, C94, C95: 10uF, Capacitor_SMD:CP_Elec_4x5.8, symbol Device:C_Polarized_US
- added C62: 10uF, Capacitor_SMD:C_0805_2012Metric, symbol Device:C
- added C63, C64: 1uF, Capacitor_SMD:C_0805_2012Metric, symbol Device:C
- added C65: 4.7uF, Capacitor_SMD:C_0805_2012Metric, symbol Device:C
- added C66: 2.2uF, Capacitor_SMD:C_0805_2012Metric, symbol Device:C
- added C76, C83, C96, C97, C98, C99: 0.1uF, Capacitor_SMD:C_0805_2012Metric, symbol Device:C
- added J10, J11, J12, J13, J3, J7, J9: AudioJack2, symbol Connector_Audio:AudioJack2
- added R100, R101, R78, R79, R86, R87, R94, R95, R96, R97, R98, R99: 10k, Resistor_SMD:R_0805_2012Metric, symbol Device:R
- added R102, R103, R104, R105, R80, R88: 1k, Resistor_SMD:R_0805_2012Metric, symbol Device:R
- added R106, R107, R108, R109, R81, R89: 270, Resistor_SMD:R_0805_2012Metric, symbol Device:R
- added R110, R111, R112, R113, R115, R117, R119, R121, R82, R84, R90, R92: 2.49k, Resistor_SMD:R_0805_2012Metric, symbol Device:R
- added R114, R116, R118, R120, R122, R123, R124, R125, R83, R85, R91, R93: 40.2, Resistor_SMD:R_0805_2012Metric, symbol Device:R
- added R76: 249k, Resistor_SMD:R_0603_1608Metric, symbol Device:R
- added R77: 499k, Resistor_SMD:R_0603_1608Metric, symbol Device:R
- added U14, U15, U19, U20, U21, U22, U23: OPA2134, symbol Amplifier_Operational:OPA2134
- added U18: LM27761, Package_SON:WSON-8-1EP_2x2mm_P0.5mm_EP0.9x1.6mm, symbol Regulator_SwitchedCapacitor:LM27761
- C52: value 1nF -> 0.1uF; footprint Capacitor_SMD:C_0402_1005Metric -> Capacitor_SMD:C_0805_2012Metric
- C53: value 100uF -> 1nF; footprint Capacitor_SMD:C_0805_2012Metric -> Capacitor_SMD:C_0402_1005Metric
- C71: value 0.1uF -> 100pF
- C75: value 1uF -> 10uF
- R57: value 1k -> 10k; footprint Resistor_SMD:R_0402_1005Metric -> Resistor_SMD:R_0805_2012Metric
- R58: value 2M2 -> 10k; footprint Resistor_SMD:R_0402_1005Metric -> Resistor_SMD:R_0805_2012Metric
- R59: value 2M2 -> 1k; footprint Resistor_SMD:R_0402_1005Metric -> Resistor_SMD:R_0805_2012Metric
- R61: value 6k8 -> 270; footprint Resistor_SMD:R_0402_1005Metric -> Resistor_SMD:R_0805_2012Metric
- R62: value 22k -> 2.49k; footprint Resistor_SMD:R_0402_1005Metric -> Resistor_SMD:R_0805_2012Metric
- R63: value 12k -> 40.2; footprint Resistor_SMD:R_0402_1005Metric -> Resistor_SMD:R_0805_2012Metric
- R64: value 1k -> 2.49k; footprint Resistor_SMD:R_0402_1005Metric -> Resistor_SMD:R_0805_2012Metric
- R65: value 1k -> 40.2; footprint Resistor_SMD:R_0402_1005Metric -> Resistor_SMD:R_0805_2012Metric
- R68: value 2.49k -> 1k
- R69: value 2.49k -> 270
- R70: value 40.2 -> 2.49k
- R72: value 270 -> 2.49k
- R73: value 1k -> 40.2
Connections:
- net -5V is gone; now on net -5V_1: C59.2, R74.1, U17.4 (VOUT)
- net A_L_5 is gone; now on net DGND: C75.2
- net IN is gone; now on an unnamed net: R57.2
- net IN_AA_BUF_IN is gone; now on an unnamed net: R63.1
- net IN_AA_BUF_OUT is gone; now on an unnamed net: R64.2
- net IN_BUF_OUT is gone; now on an unnamed net: R61.2
- net 3.3V: no longer C69.2
- net 5V: now also R57.1, C62.2, C63.2, R100.1, R78.1, R86.1, R94.1, R96.1, R98.1, U14.8 (V+), U15.8 (V+), U18.1 (VIN), U18.6 (EN), U19.8 (V+), U20.8 (V+), U21.8 (V+), U22.8 (V+), U23.8 (V+)
- net ADC1_IN+: now also C56.2, IC1.1 (VIN+), R65.2; no longer C54.2, R70.2
- net ADC1_IN-: now also C54.1, IC1.2 (VIN-), R63.2; no longer C56.1, R71.2
- net AGND: now also J10.S, J11.S, J12.S, J13.S, J3.S, J7.S, J9.S; no longer C69.1, C71.2
- net DGND: now also C52.1, C54.2, C56.1, C69.1, C71.2, R58.2, C125.2, C127.1, C128.2, C130.1, C131.2, C133.1, C134.2, C136.1, C51.2, C62.1, C63.1, C65.1, C66.1, C68.2, C73.1, C76.1, C78.2, C80.1, C82.2, C83.1, C85.2, C87.1, C92.2, C93.2, C94.2, C95.2, C96.1, C97.1, C98.1, C99.1, R101.2, R77.2, R79.2, R87.2, R95.2, R97.2, R99.2, U18.2 (GND), U18.9 (PAD); no longer C54.1, C56.2
- net at U16.3 (+), U16.5 (+): now also C75.1, C76.2, R78.2, R79.1; no longer R66.2, R67.1
- net at R62.1: now also C53.1, U14.1; no longer R63.2
- net at R61.1: now also C53.2, R59.2, U14.2 (-); no longer R62.2
- net at R68.2, R69.1: now also C70.2, U15.2 (-); no longer U16.6 (-)
- net at R73.1: now also R72.2, U15.7; no longer C53.1
- net at J5.T: now also C67.2; no longer C53.2
- net at R69.2, R70.1: now also R71.1, C70.1, U15.1; no longer U16.7
- net ADC2_IN-: now reaches C71.1
- net ADC2_IN-: now also R71.2, C72.2, C78.1, C79.2, C85.1, C86.2, R83.2, R91.2
- net -5V_1: now reaches U16.4 (V-)
- net -5V_1: now also U14.4 (V-), U15.4 (V-), U19.4 (V-)
- net ADC_IN+: no longer names the net of R64.1
- net ADC_IN+: now also R62.2, U14.6 (-)
- net ADC_IN-: no longer names the net of R65.1
- net ADC_IN-: now also U14.7
- net GND: no longer names the net of R58.1
- net GND: now also C52.2, C51.1, U14.3 (+), U14.5 (+)
- net IN_BUF: no longer names the net of R59.1
- net IN_BUF: now also C50.1
- removed net IN_RF: R57.1, R58.2
- removed net VCOM: R59.2, R65.2
- new net: C93.1, C97.2, R96.2, R97.1, U21.3 (+), U21.5 (+)
- new net: C122.1, R107.2, R111.1, R116.1, U21.1
- new net: C122.2, R103.2, R107.1, U21.2 (-)
- new net: R111.2, R117.1, U21.6 (-)
- new net: R117.2, R123.1, U21.7
- new net: R76.2, R77.1, U18.5 (VFB)
- new net: C77.1, R81.2, R82.1, R83.1, U16.1
- new net: C77.2, R80.2, R81.1, U16.2 (-)
- new net: C68.1, C69.2, R66.2, R67.1, U15.3 (+), U15.5 (+)
- new net: C123.1, R108.2, R112.1, R118.1, U22.1
- new net: R112.2, R119.1, U22.6 (-)
- new net: C91.1, R105.1
- new net: C124.2, R105.2, R109.1, U23.2 (-)
- new net: C89.2, J11.T
- new net: C64.1, U18.7 (C-)
- new net: C64.2, U18.8 (C+)
- new net: C95.1, C99.2, R100.2, R101.1, U23.3 (+), U23.5 (+)
- new net: C121.1, R106.2, R110.1, R114.1, U20.1
- new net: R110.2, R115.1, U20.6 (-)
- new net: C50.2, J3.T
- new net: R90.2, R92.1, U19.6 (-)
- new net: R92.2, R93.1, U19.7
- new net: C124.1, R109.2, R113.1, R120.1, U23.1
- new net: R70.2, R72.1, U15.6 (-)
- new net: C88.2, J10.T
- new net: C90.2, J12.T
- new net: C89.1, R103.1
- new net: C82.1, C83.2, R86.2, R87.1, U19.3 (+), U19.5 (+)
- new net: C88.1, R102.1
- new net: C81.1, R88.1
- new net: C84.2, R88.2, R89.1, U19.2 (-)
- new net: C94.1, C98.2, R98.2, R99.1, U22.3 (+), U22.5 (+)
- new net: R119.2, R124.1, U22.7
- new net: C84.1, R89.2, R90.1, R91.1, U19.1
- new net: C65.2, U18.3 (CPOUT)
- new net: C91.2, J13.T
- new net: C81.2, J9.T
- new net: C121.2, R102.2, R106.1, U20.2 (-)
- new net: R113.2, R121.1, U23.6 (-)
- new net: R121.2, R125.1, U23.7
- new net: C90.1, R104.1
- new net: C123.2, R104.2, R108.1, U22.2 (-)
- new net: R115.2, R122.1, U20.7
- new net: C92.1, C96.2, R94.2, R95.1, U20.3 (+), U20.5 (+)
- new net: R82.2, R84.1, U16.6 (-)
- new net: R84.2, R85.1, U16.7
- new net: C67.1, R68.1
- new net: C74.1, R80.1
- new net: C74.2, J7.T
- new net -5V_2: C66.2, R76.1, U18.4 (VOUT), U20.4 (V-), U21.4 (V-), U22.4 (V-), U23.4 (V-)
- new net ADC2_IN+: C72.1, C73.2, C79.1, C80.2, C86.1, C87.2, R73.2, R85.2, R93.2
- new net ADC5_IN+: C132.1, C133.2, R124.2
- new net ADC5_IN-: C131.1, C132.2, R118.2
- new net ADC6_IN+: C135.1, C136.2, R125.2
- new net ADC6_IN-: C134.1, C135.2, R120.2
- new net ADC7_IN+: C126.1, C127.2, R122.2
- new net ADC7_IN-: C125.1, C126.2, R114.2
- new net ADC8_IN+: C129.1, C130.2, R123.2
- new net ADC8_IN-: C128.1, C129.2, R116.2
Other:
- note added: "4 of the LM27761's go to the first inverter, the other 4 go to the second one."
- note added: "Buffers for each ADC's Inputs"
- note added: "Voltage Inverter w/ Max current output of 250mA Each OPA2134 uses 38mA max current, meaning for the 9 being used with dual supplies we need 2 LM27761s."
- note added: "Voltage Inverters for OPA2134's"
- note removed: "3rd order Butterworth anti-aliasing (low-pass filter) fc=25kHz"
- note removed: "ADC"
- note removed: "BNC connector"
- note removed: "Both ADC inputs should be at same VCOM"
- note removed: "HP filter: fc=1.4Hz"
- note removed: "Input voltage must be in -1.65V to +1.65V range!"
- note removed: "MCP6001: I/O Rail-to-Rail, Single-Supply (1V8 to 5V), high-impedance input CMOS, low bias currents, unity gain stable"
- note removed: "RF filter: fc=1.1MHz"
- note removed: "Rin = 1.1M"
- note removed: "Single-ended to 'balanced' conversion"
- moved on the sheet: C36, C37, C38, C39, C40, C41, C57, C58, C59, C60, C61, IC1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

Commit message: Added 3.3V/1.8V LDO, clock IC
Parts:
- removed C121, C122, C123, C124, C53, C70, C77, C84: 1nF, Capacitor_SMD:C_0402_1005Metric, symbol Device:C
- removed C125, C127, C128, C130, C131, C133, C134, C136, C54, C56, C71, C73, C78, C80, C85, C87: 100pF, Capacitor_SMD:C_0805_2012Metric, symbol Device:C
- removed C126, C129, C132, C135, C55, C72, C79, C86: 0.022uF, Capacitor_SMD:C_0805_2012Metric, symbol Device:C
- removed C36, C39, C41, C51, C68, C75, C82, C92, C93, C94, C95: 10uF, Capacitor_SMD:CP_Elec_4x5.8, symbol Device:C_Polarized_US
- removed C37, C38, C40, C52, C69, C76, C83, C96, C97, C98, C99: 0.1uF, Capacitor_SMD:C_0805_2012Metric, symbol Device:C
- removed C50, C67, C74, C81, C88, C89, C90, C91: 100uF, Capacitor_SMD:C_0805_2012Metric, symbol Device:C
- removed C62: 10uF, Capacitor_SMD:C_0805_2012Metric, symbol Device:C
- removed C63, C64: 1uF, Capacitor_SMD:C_0805_2012Metric, symbol Device:C
- removed C65: 4.7uF, Capacitor_SMD:C_0805_2012Metric, symbol Device:C
- removed C66: 2.2uF, Capacitor_SMD:C_0805_2012Metric, symbol Device:C
- removed IC1: PCM4201PWR, SOP65P640X120-16N, symbol SamacSys_Parts:PCM4201PWR
- removed J10, J11, J12, J13, J3, J5, J7, J9: AudioJack2, symbol Connector_Audio:AudioJack2
- removed R100, R101, R57, R58, R66, R67, R78, R79, R86, R87, R94, R95, R96, R97, R98, R99: 10k, Resistor_SMD:R_0805_2012Metric, symbol Device:R
- removed R102, R103, R104, R105, R59, R68, R80, R88: 1k, Resistor_SMD:R_0805_2012Metric, symbol Device:R
- removed R106, R107, R108, R109, R61, R69, R81, R89: 270, Resistor_SMD:R_0805_2012Metric, symbol Device:R
- removed R110, R111, R112, R113, R115, R117, R119, R121, R62, R64, R70, R72, R82, R84, R90, R92: 2.49k, Resistor_SMD:R_0805_2012Metric, symbol Device:R
- removed R114, R116, R118, R120, R122, R123, R124, R125, R63, R65, R71, R73, R83, R85, R91, R93: 40.2, Resistor_SMD:R_0805_2012Metric, symbol Device:R
- removed R76: 249k, Resistor_SMD:R_0603_1608Metric, symbol Device:R
- removed R77: 499k, Resistor_SMD:R_0603_1608Metric, symbol Device:R
- removed U14, U15, U16, U19, U20, U21, U22, U23: OPA2134, symbol Amplifier_Operational:OPA2134
- removed U18: LM27761, Package_SON:WSON-8-1EP_2x2mm_P0.5mm_EP0.9x1.6mm, symbol Regulator_SwitchedCapacitor:LM27761
- added C102, C110, C111, C114, C115, C118, C119, C32: 10uF, Capacitor_SMD:C_0805_2012Metric, symbol Device:C
- added C107, C112, C113: 0.1uF, Capacitor_SMD:C_0805_2012Metric, symbol Device:C
- added C116, C117: 2.2uF, Capacitor_SMD:C_0805_2012Metric, symbol Device:C
- added IC3: PCM1865DBT, SamacSys_Parts:SOP50P640X120-30N, symbol SamacSys_Parts:PCM1865DBT
Connections:
- net AGND: now also C107.1, C107.2, C110.1, C111.2, C112.1, C113.2, C116.1, C117.1, C32.1, C32.2, IC3.12 (DGND), IC3.26 (MD0), IC3.7 (AGND)
- net -5V_1 renamed -5V
- new net: C102.2, C110.2, C111.1, C112.2, C113.1, IC3.13 (DVDD), IC3.14 (IOVDD), IC3.8 (AVDD)
- new net: C117.2, IC3.11 (LDO)
- new net: C116.2, IC3.6 (VREF)
- new net: C114.2, IC3.1 (VINL2/VIN1M)
- new net: C119.1, IC3.27 (VINL4/VIN4M)
- new net: C118.1, IC3.29 (VINL3/VIN4P)
- new net: C115.2, IC3.3 (VINL1/VIN1P)
- new net 3.3V_LDO: C102.1
- new net ADDRESS: IC3.25 (MS/AD)
- new net AIN_1: C115.1
- new net AIN_2: C114.1
- new net AIN_3: C118.2
- new net AIN_4: C119.2
- new net BCK: IC3.17 (BCK)
- new net DATA_OUT_1: IC3.18 (DOUT)
- new net LRCK: IC3.16 (LRCK)
- new net SCKI: IC3.15 (SCKI)
- new net SCL: IC3.24 (MC/SCL)
- new net SDA: IC3.23 (MOSI/SDA)
Other:
- note added: "3.3V"
- note added: "Grounded = I2C"
- note removed: "4 of the LM27761's go to the first inverter, the other 4 go to the second one."
- note removed: "Buffers for each ADC's Inputs"
