File: Power_Supplies/untitled.kicad_sch (KiCad schematic)
At the start: 84 parts, among them IC2 PCM1808PWRG4, J4 XLR3, J6 XLR3_AudioJack2_Combo, J8 XLR3, SW1 SW_Push, SW2 SW_Push, SW4 SW_SPDT, SW5 SW_SPDT, SW6 SW_SPDT, U12 OPA2134, U13 SSM2019BRNZ, U6 CS4391A-KZZ, U9 MAX1044

Commit message: Added 3.3V/1.8V LDO, clock IC
Parts:
- removed C102, C107: 22uF, Capacitor_SMD:CP_Elec_4x5.8, symbol Device:C_Polarized_US
- removed C110, C112, C116: 200pF, Capacitor_SMD:C_0402_1005Metric, symbol Device:C
- removed C111, C117, C119, C120: 0.1uF, Capacitor_SMD:C_0402_1005Metric, symbol Device:C
- removed C113, C137, C32, C33: 10uF, Capacitor_SMD:CP_Elec_4x5.8, symbol Device:C_Polarized_US
- removed C114, C115: 47 uF, Capacitor_SMD:CP_Elec_4x5.8, symbol Device:C_Polarized_US
- removed C118: 0.33uF, Capacitor_SMD:C_0402_1005Metric, symbol Device:C
- removed D1, D2: LED, LED_SMD:LED_0201_0603Metric, symbol PCM_SL_Devices:LED
- removed DZ1, DZ10, DZ11, DZ12, DZ2, DZ3, DZ4, DZ9: 10V, Diode_SMD:D_SMB, symbol PCM_Diode_Zener_AKL:D_Zener_Generic
- removed J6: XLR3_AudioJack2_Combo, SamacSys_Parts:FA-238_EPS, symbol Connector_Audio:XLR3_AudioJack2_Combo
- removed J8: XLR3, symbol Connector_Audio:XLR3
- removed R30, R46, R50, R51, R52, R60: 2.2k, Resistor_SMD:R_0805_2012Metric, symbol Device:R
- removed R31, R32, R47, R48: 5.1k, Resistor_SMD:R_0805_2012Metric, symbol Device:R
- removed R33, R45: 10, Resistor_SMD:R_0805_2012Metric, symbol Device:R
- removed R49: 1M, Resistor_SMD:R_0805_2012Metric, symbol Device:R
- removed R53, R54: 2.2K, Resistor_SMD:R_0805_2012Metric, symbol Device:R
- removed R55: 330, Resistor_SMD:R_0805_2012Metric, symbol Device:R
- removed R56: 22K, Resistor_SMD:R_0805_2012Metric, symbol Device:R
- removed RV1, RV2: 10k, Potentiometer_THT:Potentiometer_ACP_CA9-V10_Vertical, symbol Device:R_Potentiometer
- removed SW1, SW2: SW_Push, Button_Switch_THT:SW_PUSH_1P1T_6x3.5mm_H5.0_APEM_MJTP1250, symbol Switch:SW_Push
- removed U12: OPA2134, Package_SO:SOIC-8_3.9x4.9mm_P1.27mm, symbol Amplifier_Operational:OPA2134
- removed U13: SSM2019BRNZ, SamacSys_Parts:SOIC127P600X175-8N, symbol SDLibrary:SSM2019BRNZ
- removed U9: MAX1044, SamacSys_Parts:SOIC127P600X175-8N, symbol Regulator_SwitchedCapacitor:MAX1044
- added C121, C122, C123, C124, C72, C73, C74, C75: 1nF, Capacitor_SMD:C_0402_1005Metric, symbol Device:C
- added C125, C127, C128, C130, C131, C133, C134, C136, C76, C78, C79, C81, C82, C84, C85, C87: 100pF, Capacitor_SMD:C_0805_2012Metric, symbol Device:C
- added C126, C129, C132, C135, C77, C80, C83, C86: 0.022uF, Capacitor_SMD:C_0805_2012Metric, symbol Device:C
- added C153, C154, C36, C40, C41, C64, C65, C66, C67, C92, C93, C94, C95: 10uF, Capacitor_SMD:CP_Elec_4x5.8, symbol Device:C_Polarized_US
- added C37, C38, C39, C68, C69, C70, C71, C96, C97, C98, C99: 0.1uF, Capacitor_SMD:C_0805_2012Metric, symbol Device:C
- added C50, C51: 10uF, Capacitor_SMD:C_0805_2012Metric, symbol Device:C
- added C52, C53, C54, C55: 1uF, Capacitor_SMD:C_0805_2012Metric, symbol Device:C
- added C56, C57: 4.7uF, Capacitor_SMD:C_0805_2012Metric, symbol Device:C
- added C58, C59: 2.2uF, Capacitor_SMD:C_0805_2012Metric, symbol Device:C
- added C60, C61, C62, C63, C88, C89, C90, C91: 100uF, Capacitor_SMD:C_0805_2012Metric, symbol Device:C
- added IC1: PCM4201PWR, SOP65P640X120-16N, symbol SamacSys_Parts:PCM4201PWR
- added J10, J11, J12, J13, J3, J5, J7, J9: AudioJack2, symbol Connector_Audio:AudioJack2
- added R100, R101, R62, R63, R64, R65, R66, R67, R68, R69, R94, R95, R96, R97, R98, R99: 10k, Resistor_SMD:R_0805_2012Metric, symbol Device:R
- added R102, R103, R104, R105, R70, R71, R72, R73: 1k, Resistor_SMD:R_0805_2012Metric, symbol Device:R
- added R106, R107, R108, R109, R74, R75, R76, R77: 270, Resistor_SMD:R_0805_2012Metric, symbol Device:R
- added R110, R111, R112, R113, R115, R117, R119, R121, R78, R79, R80, R81, R83, R85, R87, R89: 2.49k, Resistor_SMD:R_0805_2012Metric, symbol Device:R
- added R114, R116, R118, R120, R122, R123, R124, R125, R82, R84, R86, R88, R90, R91, R92, R93: 40.2, Resistor_SMD:R_0805_2012Metric, symbol Device:R
- added R57, R59: 249k, Resistor_SMD:R_0603_1608Metric, symbol Device:R
- added R58, R61: 499k, Resistor_SMD:R_0603_1608Metric, symbol Device:R
- added U14, U15: LM27761, Package_SON:WSON-8-1EP_2x2mm_P0.5mm_EP0.9x1.6mm, symbol Regulator_SwitchedCapacitor:LM27761
- added U16, U17, U18, U19, U20, U21, U22, U23: OPA2134, symbol Amplifier_Operational:OPA2134
- added U25: NCP1117-5.0_SOT223, Package_TO_SOT_SMD:SOT-223-3_TabPin2, symbol Regulator_Linear:NCP1117-5.0_SOT223
Connections:
- net 3.3V: now also C39.2, C41.2, IC1.13 (VDD)
- net 5V: now also C50.2, C51.2, C52.2, C53.2, R100.1, R62.1, R64.1, R66.1, R68.1, R94.1, R96.1, R98.1, U14.1 (VIN), U14.6 (EN), U15.1 (VIN), U15.6 (EN), U16.8 (V+), U17.8 (V+), U18.8 (V+), U19.8 (V+), U20.8 (V+), U21.8 (V+), U22.8 (V+), U23.8 (V+)
- net AGND: now also C153.2, C154.2, C36.2, C37.1, C38.2, C40.2, IC1.15 (VREF-), IC1.3 (AGND), J10.S, J11.S, J12.S, J13.S, J3.S, J5.S, J7.S, J9.S, U25.1 (GND)
- net DATA_BIT_CLOCK: now also IC1.11 (BCK)
- net D_OUT_1: now also IC1.9 (DATA)
- net MCLK: now also IC1.12 (SCKI)
- new net: C62.1, R72.1
- new net: C62.2, J7.T
- new net: R110.2, R115.1, U20.6 (-)
- new net: R115.2, R122.1, U20.7
- new net: C121.1, R106.2, R110.1, R114.1, U20.1
- new net: C75.1, R77.2, R81.1, R88.1, U19.1
- new net: C92.1, C96.2, R94.2, R95.1, U20.3 (+), U20.5 (+)
- new net: R87.2, R92.1, U18.7
- new net: C89.1, R103.1
- new net: C89.2, J11.T
- new net: C95.1, C99.2, R100.2, R101.1, U23.3 (+), U23.5 (+)
- new net: C124.1, R109.2, R113.1, R120.1, U23.1
- new net: C123.1, R108.2, R112.1, R118.1, U22.1
- new net: C74.1, R76.2, R80.1, R86.1, U18.1
- new net: R80.2, R87.1, U18.6 (-)
- new net: R78.2, R83.1, U16.6 (-)
- new net: R83.2, R90.1, U16.7
- new net: C65.1, C69.2, R64.2, R65.1, U17.3 (+), U17.5 (+)
- new net: C67.1, C71.2, R68.2, R69.1, U19.3 (+), U19.5 (+)
- new net: C61.1, R71.1
- new net: C73.2, R71.2, R75.1, U17.2 (-)
- new net: C63.1, R73.1
- new net: C63.2, J9.T
- new net: C122.2, R103.2, R107.1, U21.2 (-)
- new net: C122.1, R107.2, R111.1, R116.1, U21.1
- new net: R81.2, R89.1, U19.6 (-)
- new net: R89.2, R93.1, U19.7
- new net: C60.1, R70.1
- new net: C60.2, J3.T
- new net: C56.2, U14.3 (CPOUT)
- new net: R57.2, R58.1, U14.5 (VFB)
- new net: C54.1, U14.7 (C-)
- new net: C54.2, U14.8 (C+)
- new net: C66.1, C70.2, R66.2, R67.1, U18.3 (+), U18.5 (+)
- new net: C93.1, C97.2, R96.2, R97.1, U21.3 (+), U21.5 (+)
- new net: C73.1, R75.2, R79.1, R84.1, U17.1
- new net: R111.2, R117.1, U21.6 (-)
- new net: C64.1, C68.2, R62.2, R63.1, U16.3 (+), U16.5 (+)
- new net: C91.1, R105.1
- new net: C124.2, R105.2, R109.1, U23.2 (-)
- new net: C121.2, R102.2, R106.1, U20.2 (-)
- new net: C88.1, R102.1
- new net: C88.2, J10.T
- new net: R117.2, R123.1, U21.7
- new net: C55.1, U15.7 (C-)
- new net: C55.2, U15.8 (C+)
- new net: C38.1, C40.1, IC1.16 (VREF+)
- new net: C91.2, J13.T
- new net: C90.1, R104.1
- new net: C123.2, R104.2, R108.1, U22.2 (-)
- new net: C75.2, R73.2, R77.1, U19.2 (-)
- new net: R85.2, R91.1, U17.7
- new net: C57.2, U15.3 (CPOUT)
- new net: R59.2, R61.1, U15.5 (VFB)
- new net: C72.2, R70.2, R74.1, U16.2 (-)
- new net: C72.1, R74.2, R78.1, R82.1, U16.1
- new net: C74.2, R72.2, R76.1, U18.2 (-)
- new net: C94.1, C98.2, R98.2, R99.1, U22.3 (+), U22.5 (+)
- new net: C61.2, J5.T
- new net: R112.2, R119.1, U22.6 (-)
- new net: R119.2, R124.1, U22.7
- new net: R113.2, R121.1, U23.6 (-)
- new net: R121.2, R125.1, U23.7
- new net: R79.2, R85.1, U17.6 (-)
- new net: C90.2, J12.T
- new net -5V_1: C58.2, R57.1, U14.4 (VOUT), U16.4 (V-), U17.4 (V-), U18.4 (V-), U19.4 (V-)
- new net -5V_2: C59.2, R59.1, U15.4 (VOUT), U20.4 (V-), U21.4 (V-), U22.4 (V-), U23.4 (V-)
- new net 15V: C153.1, U25.3 (VI)
- new net 5V_LDO: C154.1, C36.1, C37.2, IC1.4 (VCC), U25.2 (VO)
- new net ADC1_IN+: C83.1, C84.2, IC1.1 (VIN+), R92.2
- new net ADC1_IN-: C82.1, C83.2, IC1.2 (VIN-), R86.2
- new net ADC2_IN+: C77.1, C78.2, C80.1, C81.2, C86.1, C87.2, R90.2, R91.2, R93.2
- new net ADC2_IN-: C76.1, C77.2, C79.1, C80.2, C85.1, C86.2, R82.2, R84.2, R88.2
- new net ADC5_IN+: C132.1, C133.2, R124.2
- new net ADC5_IN-: C131.1, C132.2, R118.2
- new net ADC6_IN+: C135.1, C136.2, R125.2
- new net ADC6_IN-: C134.1, C135.2, R120.2
- new net ADC7_IN+: C126.1, C127.2, R122.2
- new net ADC7_IN-: C125.1, C126.2, R114.2
- new net ADC8_IN+: C129.1, C130.2, R123.2
- new net ADC8_IN-: C128.1, C129.2, R116.2
- new net DGND: C125.2, C127.1, C128.2, C130.1, C131.2, C133.1, C134.2, C136.1, C39.1, C41.1, C50.1, C51.1, C52.1, C53.1, C56.1, C57.1, C58.1, C59.1, C64.2, C65.2, C66.2, C67.2, C68.1, C69.1, C70.1, C71.1, C76.2, C78.1, C79.2, C81.1, C82.2, C84.1, C85.2, C87.1, C92.2, C93.2, C94.2, C95.2, C96.1, C97.1, C98.1, C99.1, IC1.14 (DGND), R101.2, R58.2, R61.2, R63.2, R65.2, R67.2, R69.2, R95.2, R97.2, R99.2, U14.2 (GND), U14.9 (PAD), U15.2 (GND), U15.9 (PAD)
- new net HPFD: IC1.8 (HPFD)
- new net RATE: IC1.5 (RATE)
- new net RESET: IC1.7 (~{RST})
- new net SYNC_CLOCK: IC1.10 (FSYNC)
- new net S/M: IC1.6 (S/~{M})
Other:
- note added: "4 of the LM27761's go to the first inverter, the other 4 go to the second one."
- note added: "5V Output from LDO"
- note added: "Active High"
- note added: "Active Low"
- note added: "Buffers for each ADC's Inputs"
- note added: "NCP1117ST50T3G LDO for low noise output voltage"
- note added: "Voltage Inverter w/ Max current output of 250mA Each OPA2134 uses 38mA max current, meaning for the 9 being used with dual supplies we need 2 LM27761s."
- note added: "Voltage Inverters for OPA2134's"
- note removed: "470 pFs For RF Protection"
- note removed: "Add V/2 Offset"
- note removed: "Coupling capacitor to bring back to real ground"
- note removed: "Mic Preamp Front-end (Phantom Power)"
- note removed: "Negative"
- note removed: "Old voltage inverter (needed more current output)"
- note removed: "Phantom Power Circuit"
- note removed: "Place caps close as possible to input pins"
- note removed: "Positive"
- note removed: "Preamp Hi-Z Stage (Impedance Buffer)"
- note removed: "Preamp Mic Stage"
- note removed: "Preamp Summing Stage"
- note removed: "Provides 30 dB gain"
- note removed: "To Mic Preamp"
