File: Power_Supplies/untitled.kicad_sch (KiCad schematic)
At the start: 194 parts, among them IC1 PCM4201PWR, IC2 PCM1808PWRG4, J10 AudioJack2, J11 AudioJack2, J12 AudioJack2, J13 AudioJack2, J3 AudioJack2, J4 XLR3, J5 AudioJack2, J7 AudioJack2, J9 AudioJack2, SW4 SW_SPDT, SW5 SW_SPDT, SW6 SW_SPDT, U14 LM27761, U15 LM27761, U16 OPA2134, U17 OPA2134, U18 OPA2134, U19 OPA2134, U20 OPA2134, U21 OPA2134, U22 OPA2134, U23 OPA2134, U25 NCP1117-5.0_SOT223, U6 CS4391A-KZZ

Commit message: big things are coming...
Parts:
- added C128, C129: 10uF, Capacitor_SMD:CP_Elec_4x5.8, symbol Device:C_Polarized_US
- added U23: MAX1044, SamacSys_Parts:SOIC127P600X175-8N, symbol Regulator_SwitchedCapacitor:MAX1044
- C110: renamed from C42; now left out of the parts list
- C111: renamed from C43; now left out of the parts list
- C112: renamed from C44; now left out of the parts list
- C113: renamed from C45; now left out of the parts list
- C114: renamed from C46; now left out of the parts list
- C115: renamed from C47; now left out of the parts list
- C117: renamed from C48; now left out of the parts list
- C118: renamed from C49; now left out of the parts list
- C126: renamed from C153; now left out of the parts list
- C127: renamed from C154; now left out of the parts list
- C130: renamed from C36; now left out of the parts list
- C131: renamed from C37; now left out of the parts list
- C132: renamed from C50; now left out of the parts list
- C133: renamed from C51; now left out of the parts list
- C134: renamed from C52; now left out of the parts list
- C135: renamed from C53; now left out of the parts list
- C136: renamed from C54; now left out of the parts list
- C137: renamed from C55; now left out of the parts list
- C138: renamed from C56; now left out of the parts list
- C139: renamed from C57; now left out of the parts list
- C140: renamed from C58; now left out of the parts list
- C141: renamed from C59; now left out of the parts list
- C142: renamed from C38; now left out of the parts list
- C143: renamed from C39; now left out of the parts list
- C144: renamed from C40; now left out of the parts list
- C145: renamed from C41; now left out of the parts list
- C146: renamed from C60; now left out of the parts list
- C147: renamed from C61; now left out of the parts list
- C148: renamed from C62; now left out of the parts list
- C149: renamed from C63; now left out of the parts list
- C150: renamed from C64; now left out of the parts list
- C151: renamed from C65; now left out of the parts list
- C152: renamed from C66; now left out of the parts list
- C153: renamed from C67; now left out of the parts list
- C154: renamed from C68; now left out of the parts list
- C155: renamed from C69; now left out of the parts list
- C156: renamed from C70; now left out of the parts list
- C157: renamed from C71; now left out of the parts list
- C158: renamed from C72; now left out of the parts list
- C159: renamed from C73; now left out of the parts list
- C160: renamed from C74; now left out of the parts list
- C161: renamed from C75; now left out of the parts list
- C162: renamed from C76; now left out of the parts list
- C163: renamed from C77; now left out of the parts list
- C164: renamed from C78; now left out of the parts list
- C165: renamed from C79; now left out of the parts list
- C166: renamed from C80; now left out of the parts list
- C167: renamed from C81; now left out of the parts list
- C168: renamed from C82; now left out of the parts list
- C169: renamed from C83; now left out of the parts list
- C170: renamed from C84; now left out of the parts list
- C171: renamed from C85; now left out of the parts list
- C172: renamed from C86; now left out of the parts list
- C173: renamed from C87; now left out of the parts list
- C174: renamed from C88; now left out of the parts list
- C175: renamed from C89; now left out of the parts list
- C176: renamed from C90; now left out of the parts list
- C177: renamed from C91; now left out of the parts list
- C178: renamed from C92; now left out of the parts list
- C179: renamed from C93; now left out of the parts list
- C180: renamed from C94; now left out of the parts list
- C181: renamed from C95; now left out of the parts list
- C182: renamed from C96; now left out of the parts list
- C183: renamed from C97; now left out of the parts list
- C184: renamed from C98; now left out of the parts list
- C185: renamed from C99; now left out of the parts list
- C186: renamed from C121; now left out of the parts list
- C187: renamed from C122; now left out of the parts list
- C188: renamed from C123; now left out of the parts list
- C189: renamed from C124; now left out of the parts list
- C190: renamed from C125; now left out of the parts list
- C191: renamed from C126; now left out of the parts list
- C192: renamed from C127; now left out of the parts list
- C193: renamed from C128; now left out of the parts list
- C194: renamed from C129; now left out of the parts list
- C195: renamed from C130; now left out of the parts list
- C196: renamed from C131; now left out of the parts list
- C197: renamed from C132; now left out of the parts list
- C198: renamed from C133; now left out of the parts list
- C199: renamed from C134; now left out of the parts list
- C200: renamed from C135; now left out of the parts list
- C201: renamed from C136; now left out of the parts list
- IC3: renamed from IC2; now left out of the parts list
- IC4: renamed from IC1; now left out of the parts list
- J12: renamed from J3; now left out of the parts list
- J13: renamed from J5; now left out of the parts list
- J14: renamed from J7; now left out of the parts list
- J15: renamed from J9; now left out of the parts list
- J16: renamed from J10; now left out of the parts list
- J17: renamed from J11; now left out of the parts list
- J18: renamed from J12; now left out of the parts list
- J19: renamed from J13; now left out of the parts list
- R100: renamed from R62; now left out of the parts list
- R101: renamed from R63; now left out of the parts list
- R102: renamed from R64; now left out of the parts list
- R103: renamed from R65; now left out of the parts list
- R104: renamed from R66; now left out of the parts list
- R105: renamed from R67; now left out of the parts list
- R106: renamed from R68; now left out of the parts list
- R107: renamed from R69; now left out of the parts list
- R108: renamed from R70; now left out of the parts list
- R109: renamed from R71; now left out of the parts list
- R110: renamed from R72; now left out of the parts list
- R111: renamed from R73; now left out of the parts list
- R112: renamed from R74; now left out of the parts list
- R113: renamed from R75; now left out of the parts list
- R114: renamed from R76; now left out of the parts list
- R115: renamed from R77; now left out of the parts list
- R116: renamed from R78; now left out of the parts list
- R117: renamed from R79; now left out of the parts list
- R118: renamed from R80; now left out of the parts list
- R119: renamed from R81; now left out of the parts list
- R120: renamed from R82; now left out of the parts list
- R121: renamed from R83; now left out of the parts list
- R122: renamed from R84; now left out of the parts list
- R123: renamed from R85; now left out of the parts list
- R124: renamed from R86; now left out of the parts list
- R125: renamed from R87; now left out of the parts list
- R126: renamed from R88; now left out of the parts list
- R127: renamed from R89; now left out of the parts list
- R128: renamed from R90; now left out of the parts list
- R129: renamed from R91; now left out of the parts list
- R130: renamed from R92; now left out of the parts list
- R131: renamed from R93; now left out of the parts list
- R132: renamed from R94; now left out of the parts list
- R133: renamed from R95; now left out of the parts list
- R134: renamed from R96; now left out of the parts list
- R135: renamed from R97; now left out of the parts list
- R136: renamed from R98; now left out of the parts list
- R137: renamed from R99; now left out of the parts list
- R138: renamed from R100; now left out of the parts list
- R139: renamed from R101; now left out of the parts list
- R140: renamed from R102; now left out of the parts list
- R141: renamed from R103; now left out of the parts list
- R142: renamed from R104; now left out of the parts list
- R143: renamed from R105; now left out of the parts list
- R144: renamed from R106; now left out of the parts list
- R145: renamed from R107; now left out of the parts list
- R146: renamed from R108; now left out of the parts list
- R147: renamed from R109; now left out of the parts list
- R148: renamed from R110; now left out of the parts list
- R149: renamed from R111; now left out of the parts list
- R150: renamed from R112; now left out of the parts list
- R151: renamed from R113; now left out of the parts list
- R152: renamed from R114; now left out of the parts list
- R153: renamed from R115; now left out of the parts list
- R154: renamed from R116; now left out of the parts list
- R155: renamed from R117; now left out of the parts list
- R156: renamed from R118; now left out of the parts list
- R157: renamed from R119; now left out of the parts list
- R158: renamed from R120; now left out of the parts list
- R159: renamed from R121; now left out of the parts list
- R160: renamed from R122; now left out of the parts list
- R161: renamed from R123; now left out of the parts list
- R162: renamed from R124; now left out of the parts list
- R163: renamed from R125; now left out of the parts list
- R96: renamed from R57; now left out of the parts list
- R97: renamed from R58; now left out of the parts list
- R98: renamed from R59; now left out of the parts list
- R99: renamed from R61; now left out of the parts list
- U22: renamed from U25; now left out of the parts list
- U24: renamed from U14; now left out of the parts list
- U25: renamed from U15; now left out of the parts list
- U26: renamed from U16; now left out of the parts list
- U27: renamed from U17; now left out of the parts list
- U28: renamed from U18; now left out of the parts list
- U29: renamed from U19; now left out of the parts list
- U30: renamed from U20; now left out of the parts list
- U31: renamed from U21; now left out of the parts list
- U32: renamed from U22; now left out of the parts list
- U33: renamed from U23; now left out of the parts list
- renumbered C104 to C116, C105 to C119, C106 to C120, C14 to C121, C15 to C122, C16 to C123, C17 to C124, C18 to C125, DZ5 to DZ17, DZ6 to DZ18, DZ7 to DZ19, DZ8 to DZ20, J4 to J11, R36 to R90, R37 to R91, R38 to R92, R39 to R93, R40 to R94, R41 to R95, SW4 to SW5, SW5 to SW6, SW6 to SW7, U6 to U21
Connections:
- net 5V: now also U23.8 (V+)
- net AGND: now also C129.1, U23.3 (GND), U23.6 (LV)
- new net: C128.1, U23.2 (CAP+)
- new net: C128.2, U23.4 (CAP-)
- new net -5V: C129.2, U23.5 (VOUT)
Other:
- note added: "-5V supply rail for OPA2134"

Commit message: Added stuff for the power supply circuitry
changed all grounds to GND (same ground plane)
Parts:
- added C1, C25, C3, C9: 4.7uF, Capacitor_SMD:C_0805_2012Metric, symbol Device:C
- added C10, C2, C4: 120pF, Capacitor_SMD:C_0402_1005Metric, symbol Device:C
- added C18: 10uF, Capacitor_SMD:C_0805_2012Metric, symbol Device:C
- added C23, C24: 1uF, Capacitor_SMD:C_0805_2012Metric, symbol Device:C
- added C26: 2.2uF, Capacitor_SMD:C_0805_2012Metric, symbol Device:C
- added C5, Cout1, Cout2, Cout3, Cout4, Cout6: 22uF, Capacitor_SMD:C_0805_2012Metric, symbol Device:C
- added C6, C8: 10uF, Capacitor_SMD:CP_Elec_4x5.8, symbol Device:C_Polarized_US
- added C7: 430pF, Capacitor_SMD:C_0402_1005Metric, symbol Device:C
- added Cout5: 47uF, Capacitor_SMD:C_0805_2012Metric, symbol Device:C
- added L1, L2, L3: 470nH, Inductor_SMD:L_0805_2012Metric, symbol Device:L
- added R1: 20k, Resistor_SMD:R_0805_2012Metric, symbol Device:R
- added R10: 523k, Resistor_SMD:R_0805_2012Metric, symbol Device:R
- added R11, R5, R9, Rpg1, Rpg2, Rpg3: 100k, Resistor_SMD:R_0805_2012Metric, symbol Device:R
- added R12: 10k, PCM_Resistor_SMD_AKL:R_0805_2012Metric_Pad1.15x1.40mm_HandSolder, symbol Device:R
- added R13: 49.9k, PCM_Resistor_SMD_AKL:R_0805_2012Metric_Pad1.15x1.40mm_HandSolder, symbol Device:R
- added R14, Rpg4: 100k, PCM_Resistor_SMD_AKL:R_0805_2012Metric_Pad1.15x1.40mm_HandSolder, symbol Device:R
- added R15: 249k, Resistor_SMD:R_0603_1608Metric, symbol Device:R
- added R16: 499k, Resistor_SMD:R_0603_1608Metric, symbol Device:R
- added R2: 52.3k, Resistor_SMD:R_0805_2012Metric, symbol Device:R
- added R3: 30.1k, Resistor_SMD:R_0805_2012Metric, symbol Device:R
- added R4: 453k, Resistor_SMD:R_0805_2012Metric, symbol Device:R
- added R6: 28k, Resistor_SMD:R_0805_2012Metric, symbol Device:R
- added R7: 56.2k, Resistor_SMD:R_0805_2012Metric, symbol Device:R
- added R8: 200k, Resistor_SMD:R_0805_2012Metric, symbol Device:R
- added U1, U3, U7: TPS62822DLC, Package_SON:Texas_VSON-HR-8_1.5x2mm_P0.5mm, symbol Regulator_Switching:TPS62822DLC
- added U2, U4: TPS73601DBV, Package_TO_SOT_SMD:SOT-23-5, symbol Regulator_Linear:TPS73601DBV
- added U5: NCP1117-5.0_SOT223, Package_TO_SOT_SMD:SOT-223-3_TabPin2, symbol Regulator_Linear:NCP1117-5.0_SOT223
- added U6: TPS82140, Package_LGA:Texas_SIL0008D_MicroSiP-8-1EP_2.8x3mm_P0.65mm_EP1.1x1.9mm_ThermalVias, symbol Regulator_Switching:TPS82140
- added U8: LM27761, Package_SON:WSON-8-1EP_2x2mm_P0.5mm_EP0.9x1.6mm, symbol Regulator_SwitchedCapacitor:LM27761
Connections:
- net -5V: now also C26.2, R15.1, U8.4 (VOUT)
- net 15V: now also C5.1, C6.1, U5.3 (VI), U6.1 (EN), U6.2 (VIN)
- net 3.3V: now also C2.1, Cout1.1, Cout2.1, Cout3.1, L1.2, R4.1
- net 5V: now also C1.1, C18.2, C23.2, C3.1, C9.1, Cout5.1, R1.1, R10.1, R12.1, Rpg1.1, Rpg2.1, Rpg3.2, Rpg4.1, U1.7 (VIN), U2.1 (IN), U2.3 (EN), U3.1 (EN), U3.7 (VIN), U4.1 (IN), U4.3 (EN), U6.4 (VOUT), U6.5 (VOUT), U7.7 (VIN), U8.1 (VIN), U8.6 (EN)
- net 5V_LDO: now also C8.1, U5.2 (VO)
- new net: C7.1, U6.8 (SS/TR)
- new net: R2.2, R3.1, U2.4 (FB)
- new net: R6.2, R7.1, U4.4 (FB)
- new net: Rpg4.2, U7.8 (PG)
- new net: R15.2, R16.1, U8.5 (VFB)
- new net: R1.2, U1.1 (EN)
- new net: C25.2, U8.3 (CPOUT)
- new net: C24.1, U8.7 (C-)
- new net: C24.2, U8.8 (C+)
- new net: Rpg2.2, U3.8 (PG)
- new net: Rpg3.1, U6.7 (PG)
- new net 0.9V: C10.1, Cout6.1, L3.2, R13.1
- new net 0.9V_EN: R12.2, Rpg1.2, U1.8 (PG), U7.1 (EN)
- new net 1.8V: C4.1, Cout4.1, L2.2, R8.1
- new net 1.8V_LDO: R6.1, U4.5 (OUT)
- new net 3.3V_LDO: R2.1, U2.5 (OUT)
- new net GND: C1.2, C18.1, C23.1, C25.1, C26.1, C3.2, C5.2, C6.2, C7.2, C8.2, C9.2, Cout1.2, Cout2.2, Cout3.2, Cout4.2, Cout5.2, Cout6.2, R11.2, R14.2, R16.2, R3.2, R5.2, R7.2, R9.2, U1.3 (AGND), U1.5 (PGND), U2.2 (GND), U3.3 (AGND), U3.5 (PGND), U4.2 (GND), U5.1 (GND), U6.3 (GND), U6.9 (GND), U7.3 (AGND), U7.5 (PGND), U8.2 (GND), U8.9 (PAD)
- new net V_Buck_0.9: L3.1, U7.6 (SW)
- new net V_Buck_1.8: L2.1, U3.6 (SW)
- new net V_Buck_3.3: L1.1, U1.6 (SW)
- new net V_FB: C2.2, R4.2, R5.1, U1.2 (FB)
- new net V_FB_0.9: C10.2, R13.2, R14.1, U7.2 (FB)
- new net V_FB_1.8: C4.2, R8.2, R9.1, U3.2 (FB)
- new net V_FB_5: R10.2, R11.1, U6.6 (FB)
Other:
- note added: "0.9V Buck Converter"
- note added: "1.8V Buck Converter"
- note added: "1.8V Output from LDO"
- note added: "1.8V output for lower noise XMOS power rail"
- note added: "3.3V Buck Converter"
- note added: "3.3V Output from LDO"
- note added: "3.3V output for lower noise ADC power rail"
- note added: "5V Output from Buck Converter"
- note added: "Vout = Vfb * (1+ R1/R2) Vfb = 0.6V Vout = 0.6 * (1+453/100) = 3.32V"
- note added: "Vout = Vfb * (1+ R3/R4) Vfb = 0.6V Vout = 0.6 * (1+200/100) = 1.8V"
- note added: "Vout = Vfb * (1+ R3/R4) Vfb = 0.6V Vout = 0.6 * (1+49.9/100) = 0.9V"
- note added: "Vout = Vfb * (1+ R5/R6) Vfb = 0.8V Vout = 0.8 * (1+523/100) = 5V"
- moved on the sheet: C126, C127, U22
