File: Power_Supplies/Power_Supplies.kicad_sch (KiCad schematic)
At the start: 0 parts

Commit message: Add files via upload
Other:
- removed sheet Preamps
- added sheet Preamp (PREAMPS.kicad_sch)
- note removed: "Preamp Circuitry"
Changed lines of the file:
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@@
 	)
 	(rectangle
-		(start 26.67 74.93)
-		(end 95.25 105.41)
+		(start 187.96 82.55)
+		(end 256.54 113.03)
 		(stroke
 			(width 0)
@@
 	)
 	(rectangle
-		(start 208.28 73.66)
-		(end 271.78 140.97)
+		(start 41.91 82.55)
+		(end 105.41 149.86)
 		(stroke
 			(width 0)
@@
 		)
 	)
-	(rectangle
-		(start 25.4 127)
-		(end 101.6 177.8)
-		(stroke
-			(width 0)
-			(type default)
-		)
-		(fill
-			(type none)
-		)
-	)
 	(text "MCUs"
 		(exclude_from_sim no)
-		(at 241.3 69.85 0)
+		(at 74.93 78.74 0)
 		(effects
 			(font
@@
 	(text "Signal Converters"
 		(exclude_from_sim no)
-		(at 58.42 72.136 0)
+		(at 219.71 79.756 0)
 		(effects
 			(font
@@
 		)
 	)
-	(text "Preamp Circuitry\n"
-		(exclude_from_sim no)
-		(at 47.752 122.936 0)
-		(effects
-			(font
-				(size 3 3)
-				(thickness 0.6)
-				(bold yes)
-				(italic yes)
-			)
-		)
-	)
 	(hierarchical_label "5V_IN"
 		(shape input)
@@
 	)
 	(sheet
-		(at 67.31 81.28)
+		(at 228.6 88.9)
 		(size 24.13 15.24)
 		(fields_autoplaced yes)
@@
 		)
 		(property "Sheetname" "DACs"
-			(at 67.31 80.5684 0)
+			(at 228.6 88.1884 0)
 			(effects
 				(font
@@
 		)
 		(property "Sheetfile" "DAC.kicad_sch"
-			(at 67.31 97.1046 0)
+			(at 228.6 104.7246 0)
 			(effects
 				(font
@@
 	)
 	(sheet
-		(at 215.9 77.47)
+		(at 49.53 86.36)
 		(size 40.64 22.86)
 		(fields_autoplaced yes)
@@
 		)
 		(property "Sheetname" "Xcore"
-			(at 215.9 76.7584 0)
+			(at 49.53 85.6484 0)
 			(effects
 				(font
@@
 		)
 		(property "Sheetfile" "XCORE.kicad_sch"
-			(at 215.9 100.9146 0)
+			(at 49.53 109.8046 0)
 			(effects
 				(font
@@
 	)
 	(sheet
-		(at 46.99 35.56)
+		(at 33.02 33.02)
 		(size 24.13 16.51)
 		(fields_autoplaced yes)
@@
 		)
 		(property "Sheetname" "Phantom Power"
-			(at 46.99 34.8484 0)
+			(at 33.02 32.3084 0)
 			(effects
 				(font
@@
 		)
 		(property "Sheetfile" "Phantom.kicad_sch"
-			(at 46.99 52.6546 0)
+			(at 33.02 50.1146 0)
 			(effects
 				(font
@@
 		)
 		(property "Field2" ""
-			(at 46.99 35.56 0)
+			(at 33.02 33.02 0)
 			(effects
 				(font
@@
 	)
 	(sheet
-		(at 29.21 81.28)
+		(at 190.5 88.9)
 		(size 24.13 15.24)
 		(fields_autoplaced yes)
@@
 		)
 		(property "Sheetname" "ADCs"
-			(at 29.21 80.5684 0)
+			(at 190.5 88.1884 0)
 			(effects
 				(font
@@
 		)
 		(property "Sheetfile" "ADC.kicad_sch"
-			(at 29.21 97.1046 0)
+			(at 190.5 104.7246 0)
 			(effects
 				(font
@@
 	)
 	(sheet
-		(at 31.75 140.97)
-		(size 25.4 25.4)
-		(fields_autoplaced yes)
-		(stroke
-			(width 0.1524)
-			(type solid)
-		)
-		(fill
-			(color 0 0 0 0.0000)
-		)
-		(property "Sheetname" "Preamps"
-			(at 31.75 140.2584 0)
-			(effects
-				(font
-					(size 1.27 1.27)
-				)
-				(justify left bottom)
-			)
-		)
-		(property "Sheetfile" "PREAMPS.kicad_sch"
-			(at 31.75 166.9546 0)
-			(effects
-				(font
-					(size 1.27 1.27)
-				)
-				(justify left top)
-			)
-		)
-		(instances
-			(project "Power_Supplies"
-				(path "/5266cf9e-da90-4c53-80fd-cf3dbed42632"
-					(page "11")
-				)
-			)
-		)
-	)
-	(sheet
 		(at 158.75 30.48)
 		(size 68.58 5.08)
@@
 	)
 	(sheet
-		(at 127 175.26)
+		(at 64.77 33.02)
+		(size 16.51 16.51)
+		(fields_autoplaced yes)
+		(stroke
+			(width 0.1524)
+			(type solid)
+		)
+		(fill
+			(color 0 0 0 0.0000)
+		)
+		(property "Sheetname" "Preamp"
+			(at 64.77 32.3084 0)
+			(effects
+				(font
+					(size 1.27 1.27)
+				)
+				(justify left bottom)
+			)
+		)
+		(property "Sheetfile" "PREAMPS.kicad_sch"
+			(at 64.77 50.1146 0)
+			(effects
+				(font
+					(size 1.27 1.27)
+				)
+				(justify left top)
+			)
+		)
+		(instances
+			(project "Power_Supplies"
+				(path "/5266cf9e-da90-4c53-80fd-cf3dbed42632"
+					(page "11")
+				)
+			)
+		)
+	)
+	(sheet
+		(at 236.22 143.51)
 		(size 45.72 17.78)
 		(fields_autoplaced yes)
@@
 		)
 		(property "Sheetname" "recycle bin"
-			(at 127 174.5484 0)
+			(at 236.22 142.7984 0)
 			(effects
 				(font
@@
 		)
 		(property "Sheetfile" "untitled.kicad_sch"
-			(at 127 193.6246 0)
-			(effects
-				(font
-					(size 1.27 1.27)
-				)
-				(justify left top)
-			)
-		)
-		(instances
-			(project "Power_Supplies"
-				(path "/5266cf9e-da90-4c53-80fd-cf3dbed42632"
-					(page "8")
-				)
-			)
+			(at 236.22 161.8746 0)
+			(effects
+				(font
+					(size 1.27 1.27)
+				)
+				(justify left top)
+			)
+		)
+		(instances
+			(project "Power_Supplies"
+				(path "/5266cf9e-da90-4c53-80fd-cf3dbed42632"
+					(page "11")
+				)
+			)

Commit message: big things are coming...
Changed lines of the file:
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@@
 		(company "Michael Meyers")
-	)
-	(junction
-		(at 144.78 41.91)
-		(diameter 0)
-		(color 0 0 0 0)
-	)
-	(junction
-		(at 144.78 45.72)
-		(diameter 0)
-		(color 0 0 0 0)
-	)
-	(wire
-		(pts
-			(xy 144.78 45.72) (xy 144.78 57.15)
-		)
-		(stroke
-			(width 0)
-			(type default)
-		)
-	)
-	(wire
-		(pts
-			(xy 144.78 57.15) (xy 158.75 57.15)
-		)
-		(stroke
-			(width 0)
-			(type default)
-		)
-	)
-	(wire
-		(pts
-			(xy 144.78 41.91) (xy 144.78 45.72)
-		)
-		(stroke
-			(width 0)
-			(type default)
-		)
-	)
-	(wire
-		(pts
-			(xy 227.33 33.02) (xy 238.76 33.02)
-		)
-		(stroke
-			(width 0)
-			(type default)
-		)
-	)
-	(wire
-		(pts
-			(xy 158.75 45.72) (xy 144.78 45.72)
-		)
-		(stroke
-			(width 0)
-			(type default)
-		)
-	)
-	(wire
-		(pts
-			(xy 125.73 41.91) (xy 144.78 41.91)
-		)
-		(stroke
-			(width 0)
-			(type default)
-		)
-	)
-	(wire
-		(pts
-			(xy 144.78 33.02) (xy 144.78 41.91)
-		)
-		(stroke
-			(width 0)
-			(type default)
-		)
-	)
-	(wire
-		(pts
-			(xy 238.76 33.02) (xy 238.76 57.15)
-		)
-		(stroke
-			(width 0)
-			(type default)
-		)
-	)
-	(wire
-		(pts
-			(xy 238.76 57.15) (xy 227.33 57.15)
-		)
-		(stroke
-			(width 0)
-			(type default)
-		)
-	)
-	(wire
-		(pts
-			(xy 144.78 33.02) (xy 158.75 33.02)
-		)
-		(stroke
-			(width 0)
-			(type default)
-		)
 	)
 	(rectangle
