File: Power_Supplies/Phantom.kicad_sch (KiCad schematic)
At the start: 17 parts, among them IC2 LT8338, U37 PEC11R-4030F-N0024

Commit message: Add files via upload
Parts:
- added H1, H2, H3, H4: MountingHole_M3, MountingHole:MountingHole_3.2mm_M3, symbol PCM_SL_Mechanical:MountingHole_M3
- added J28: PINHD_1x2_Female, Connector_PinSocket_2.54mm:PinSocket_1x02_P2.54mm_Vertical, symbol PCM_SL_Pin_Headers:PINHD_1x2_Female
- added J34, J38, J39, J40: PINHD_1x1_Female, Connector_PinSocket_2.54mm:PinSocket_1x01_P2.54mm_Vertical, symbol PCM_SL_Pin_Headers:PINHD_1x1_Female
- added J37: PINHD_1x3_Female, Connector_PinSocket_2.54mm:PinSocket_1x03_P2.54mm_Vertical, symbol PCM_SL_Pin_Headers:PINHD_1x3_Female
Connections:
- net 12V: now also J38.1
- net 5V: now also J40.1
- net at C235.1, R178.2, U37.B1 (CHANNEL_2): now also J28.2
- net at C234.2, R177.2, U37.A1 (CHANNEL_1): now also J28.1
- net AGND renamed GND
- net GND: now also J34.1
- new net -12V: J39.1
- new net 0.9V: J37.2
- new net 1.8V: J37.1
- new net 3.3V: J37.3
Other:
- moved on the sheet: C234, C235, R175, R176, R177, R178
