File: Power_Supplies/Power_Supplies.kicad_pcb (KiCad board)
At the start: 2 copper layers, 84 parts, among them J1 Line Out, J2 Headphone Out, U1 TPS62822DLC, U2 TPS62822DLC, U3 TPS82140, U4 TPS62822DLC, U5 TPA6110A2DGN, U7 PCM1780, U8 OPA2134

Commit message: big things are coming...
Parts:
- added C100: 47 uF, Capacitor_SMD:CP_Elec_4x5.8, F.Cu at (218.2, 118.2)
- added C101: 47 uF, Capacitor_SMD:CP_Elec_4x5.8, F.Cu at (226.0, 106.5)
- added C102: 47 uF, Capacitor_SMD:CP_Elec_4x5.8, F.Cu at (226.0, 112.3)
- added C103: 47 uF, Capacitor_SMD:CP_Elec_4x5.8, F.Cu at (226.0, 118.2)
- added C104: 200pF, Capacitor_SMD:C_0402_1005Metric, F.Cu at (238.2, 62.6)
- added C105: 200pF, Capacitor_SMD:C_0402_1005Metric, F.Cu at (238.2, 64.6)
- added C106: 0.1uF, Capacitor_SMD:C_0402_1005Metric, F.Cu at (238.2, 66.6)
- added C107: 0.1uF, Capacitor_SMD:C_0402_1005Metric, F.Cu at (238.2, 68.6)
- added C108: 0.1uF, Capacitor_SMD:C_0402_1005Metric, F.Cu at (238.2, 70.5)
- added C109: 0.1uF, Capacitor_SMD:C_0402_1005Metric, F.Cu at (238.2, 72.5)
- added C36: 120pF, Capacitor_SMD:C_0402_1005Metric, F.Cu at (261.9, 88.0)
- added C37: 0.1uF, Capacitor_SMD:C_0805_2012Metric, F.Cu at (254.7, 59.2)
- added C38: 10uF, Capacitor_SMD:CP_Elec_4x5.8, F.Cu at (248.6, 60.6)
- added C39: 10uF, Capacitor_SMD:CP_Elec_4x5.8, F.Cu at (248.6, 66.5)
- added C40: 10uF, Capacitor_SMD:CP_Elec_4x5.8, F.Cu at (248.6, 72.3)
- added C41: 10uF, Capacitor_SMD:CP_Elec_4x5.8, F.Cu at (248.6, 78.2)
- added C42: 10uF, Capacitor_SMD:CP_Elec_4x5.8, F.Cu at (248.6, 84.0)
- added C43: 10uF, Capacitor_SMD:CP_Elec_4x5.8, F.Cu at (248.6, 89.9)
- added C44: 1uF, Capacitor_SMD:C_0805_2012Metric, F.Cu at (81.0, 134.0)
- added C45: 1uF, Capacitor_SMD:C_0805_2012Metric, F.Cu at (79.0, 121.0)
- added C46: 1uF, Capacitor_SMD:C_0805_2012Metric, F.Cu at (79.0, 124.0)
- added C47: 10uF, Capacitor_SMD:C_0805_2012Metric, F.Cu at (81.0, 140.0)
- added C48: 1uF, Capacitor_SMD:C_0805_2012Metric, F.Cu at (81.0, 137.0)
- added C49: 18pF, Capacitor_SMD:C_0402_1005Metric, F.Cu at (264.9, 104.7)
- added C50: 18pF, Capacitor_SMD:C_0402_1005Metric, F.Cu at (264.9, 106.6)
- added C51: 2.2uF, Capacitor_SMD:C_0402_1005Metric, F.Cu at (250.6, 127.3)
- added C52: 2.2uF, Capacitor_SMD:C_0402_1005Metric, F.Cu at (250.6, 129.3)
- added C53: 2.2uF, Capacitor_SMD:C_0402_1005Metric, F.Cu at (250.6, 131.3)
- added C54: 200pF, Capacitor_SMD:C_0402_1005Metric, F.Cu at (226.7, 58.7)
- added C55: 200pF, Capacitor_SMD:C_0402_1005Metric, F.Cu at (226.7, 60.7)
- added C56: 470pF, Capacitor_SMD:C_0402_1005Metric, F.Cu at (226.7, 62.6)
- added C57: 470pF, Capacitor_SMD:C_0402_1005Metric, F.Cu at (226.7, 64.6)
- added C58: 0.01uF, Capacitor_SMD:C_0402_1005Metric, F.Cu at (226.7, 66.6)
- added C59: 0.01uF, Capacitor_SMD:C_0402_1005Metric, F.Cu at (226.7, 68.6)
- added C60: 470pF, Capacitor_SMD:C_0402_1005Metric, F.Cu at (226.7, 70.5)
- added C61: 470pF, Capacitor_SMD:C_0402_1005Metric, F.Cu at (226.7, 72.5)
- added C62: 200pF, Capacitor_SMD:C_0402_1005Metric, F.Cu at (226.7, 74.5)
- added C63: 200pF, Capacitor_SMD:C_0402_1005Metric, F.Cu at (229.6, 58.7)
- added C64: 47uF, Capacitor_SMD:CP_Elec_4x5.8, F.Cu at (202.7, 106.5)
- added C65: 22uF, Capacitor_SMD:C_0402_1005Metric, F.Cu at (229.6, 60.7)
- added C66: 22uF, Capacitor_SMD:C_0402_1005Metric, F.Cu at (229.6, 62.6)
- added C67: 47uF, Capacitor_SMD:CP_Elec_4x5.8, F.Cu at (202.7, 112.3)
- added C68: 22uF, Capacitor_SMD:C_0402_1005Metric, F.Cu at (229.6, 64.6)
- added C69: 22uF, Capacitor_SMD:C_0402_1005Metric, F.Cu at (229.6, 66.6)
- added C70: 47 uF, Capacitor_SMD:CP_Elec_4x5.8, F.Cu at (202.7, 118.2)
- added C71: 47 uF, Capacitor_SMD:CP_Elec_4x5.8, F.Cu at (210.5, 106.5)
- added C72: 47 uF, Capacitor_SMD:CP_Elec_4x5.8, F.Cu at (210.5, 112.3)
- added C73: 47 uF, Capacitor_SMD:CP_Elec_4x5.8, F.Cu at (210.5, 118.2)
- added C74: 200pF, Capacitor_SMD:C_0402_1005Metric, F.Cu at (229.6, 68.6)
- added C75: 200pF, Capacitor_SMD:C_0402_1005Metric, F.Cu at (229.6, 70.5)
- added C76: 0.1uF, Capacitor_SMD:C_0402_1005Metric, F.Cu at (229.6, 72.5)
- added C77: 0.1uF, Capacitor_SMD:C_0402_1005Metric, F.Cu at (229.6, 74.5)
- added C78: 0.1uF, Capacitor_SMD:C_0402_1005Metric, F.Cu at (232.5, 58.7)
- added C79: 0.1uF, Capacitor_SMD:C_0402_1005Metric, F.Cu at (232.5, 60.7)
- added C80: 0.01uF, Capacitor_SMD:C_0402_1005Metric, F.Cu at (232.5, 62.6)
- added C81: 0.01uF, Capacitor_SMD:C_0402_1005Metric, F.Cu at (232.5, 64.6)
- added C82: 0.1uF, Capacitor_SMD:C_0402_1005Metric, F.Cu at (232.5, 66.6)
- added C83: 0.1uF, Capacitor_SMD:C_0402_1005Metric, F.Cu at (232.5, 68.6)
- added C84: 0.1uF, Capacitor_SMD:C_0402_1005Metric, F.Cu at (232.5, 70.5)
- added C85: 0.1uF, Capacitor_SMD:C_0402_1005Metric, F.Cu at (232.5, 72.5)
- added C86: 200pF, Capacitor_SMD:C_0402_1005Metric, F.Cu at (232.5, 74.5)
- added C87: 200pF, Capacitor_SMD:C_0402_1005Metric, F.Cu at (235.3, 58.7)
- added C88: 470pF, Capacitor_SMD:C_0402_1005Metric, F.Cu at (235.3, 60.7)
- added C89: 470pF, Capacitor_SMD:C_0402_1005Metric, F.Cu at (235.3, 62.6)
- added C90: 470pF, Capacitor_SMD:C_0402_1005Metric, F.Cu at (235.3, 64.6)
- added C91: 470pF, Capacitor_SMD:C_0402_1005Metric, F.Cu at (235.3, 66.6)
- added C92: 200pF, Capacitor_SMD:C_0402_1005Metric, F.Cu at (235.3, 68.6)
- added C93: 200pF, Capacitor_SMD:C_0402_1005Metric, F.Cu at (235.3, 70.5)
- added C94: 47uF, Capacitor_SMD:CP_Elec_4x5.8, F.Cu at (218.2, 106.5)
- added C95: 22uF, Capacitor_SMD:C_0402_1005Metric, F.Cu at (235.3, 72.5)
- added C96: 22uF, Capacitor_SMD:C_0402_1005Metric, F.Cu at (235.3, 74.5)
- added C97: 47uF, Capacitor_SMD:CP_Elec_4x5.8, F.Cu at (218.2, 112.3)
- added C98: 22uF, Capacitor_SMD:C_0402_1005Metric, F.Cu at (238.2, 58.7)
- added C99: 22uF, Capacitor_SMD:C_0402_1005Metric, F.Cu at (238.2, 60.7)
- added D1: LED, LED_SMD:LED_0201_0603Metric, F.Cu at (231.3, 104.4)
- added D2: LED, LED_SMD:LED_0201_0603Metric, F.Cu at (231.3, 106.2)
- added D3: LED, LED_SMD:LED_0201_0603Metric, F.Cu at (231.3, 107.9)
- added D4: LED, LED_SMD:LED_0201_0603Metric, F.Cu at (231.3, 109.7)
- added DZ1: 10V, Diode_SMD:D_SMB, F.Cu at (203.1, 84.1)
- added DZ10: 10V, Diode_SMD:D_SMB, F.Cu at (219.8, 89.7)
- added DZ11: 10V, Diode_SMD:D_SMB, F.Cu at (219.8, 95.2)
- added DZ12: 10V, Diode_SMD:D_SMB, F.Cu at (219.8, 100.8)
- added DZ13: 10V, Diode_SMD:D_SMB, F.Cu at (228.2, 84.1)
- added DZ14: 10V, Diode_SMD:D_SMB, F.Cu at (228.2, 89.7)
- added DZ15: 10V, Diode_SMD:D_SMB, F.Cu at (228.2, 95.2)
- added DZ16: 10V, Diode_SMD:D_SMB, F.Cu at (228.2, 100.8)
- added DZ2: 10V, Diode_SMD:D_SMB, F.Cu at (203.1, 89.7)
- added DZ3: 10V, Diode_SMD:D_SMB, F.Cu at (203.1, 95.2)
- added DZ4: 10V, Diode_SMD:D_SMB, F.Cu at (203.1, 100.8)
- added DZ5: 10V, Diode_SMD:D_SMB, F.Cu at (211.4, 84.1)
- added DZ6: 10V, Diode_SMD:D_SMB, F.Cu at (211.4, 89.7)
- added DZ7: 10V, Diode_SMD:D_SMB, F.Cu at (211.4, 95.2)
- added DZ8: 10V, Diode_SMD:D_SMB, F.Cu at (211.4, 100.8)
- added DZ9: 10V, Diode_SMD:D_SMB, F.Cu at (219.8, 84.1)
- added IC1: PCM1865DBT, SamacSys_Parts:SOP50P640X120-30N, F.Cu at (262.3, 127.1)
- added IC2: LT8338, SamacSys_Parts:SOP65P490X110-9N, F.Cu at (252.6, 124.6)
- added J10: XLR3_AudioJack3_Combo, Connector_Audio:Jack_XLR-6.35mm_Neutrik_NCJ5FI-H-0_Horizontal, F.Cu at (17.9, 31.4)
- added J20: ACJM-MV-2, SamacSys_Parts:ACJMMV2, F.Cu at (155.5, 26.7)
- added J3: XLR3_AudioJack3_Combo, Connector_Audio:Jack_XLR-6.35mm_Neutrik_NCJ5FI-H-0_Horizontal, F.Cu at (110.7, 31.3)
- added J4: XLR3_AudioJack3_Combo, Connector_Audio:Jack_XLR-6.35mm_Neutrik_NCJ5FI-H-0_Horizontal, F.Cu at (79.9, 31.4)
- added J5: ACJM-MV-2, SamacSys_Parts:ACJMMV2, F.Cu at (176.5, 26.7)
- added J6: ACJM-MV-2, SamacSys_Parts:ACJMMV2, F.Cu at (197.5, 26.7)
- added J7: ACJM-MV-2, SamacSys_Parts:ACJMMV2, F.Cu at (218.5, 26.7)
- added J9: XLR3_AudioJack3_Combo, Connector_Audio:Jack_XLR-6.35mm_Neutrik_NCJ5FI-H-0_Horizontal, F.Cu at (48.9, 31.4)
- added L4: 10uH, Inductor_SMD:L_0805_2012Metric, F.Cu at (251.4, 133.6)
- added R28: 100, Resistor_SMD:R_0805_2012Metric, F.Cu at (259.1, 59.2)
- added R29: 20k, Resistor_SMD:R_0805_2012Metric, F.Cu at (83.4, 117.9)
- added R30: 20k, Resistor_SMD:R_0805_2012Metric, F.Cu at (83.5, 120.8)
- added R31: 82k, Resistor_SMD:R_0805_2012Metric, F.Cu at (83.4, 123.8)
- added R32: 82k, Resistor_SMD:R_0805_2012Metric, F.Cu at (83.4, 126.7)
- added R33: 82k, Resistor_SMD:R_0805_2012Metric, F.Cu at (94.1, 140.0)
- added R34: 10K, Resistor_SMD:R_0805_2012Metric, F.Cu at (265.6, 96.3)
- added R35: 33, Resistor_SMD:R_0805_2012Metric, F.Cu at (265.6, 99.2)
- added R36: 1M, Resistor_SMD:R_0805_2012Metric, F.Cu at (265.6, 102.2)
- added R37: 1M, Resistor_SMD:R_0805_2012Metric, F.Cu at (246.9, 124.0)
- added R38: 162k, Resistor_SMD:R_0805_2012Metric, F.Cu at (246.9, 126.9)
- added R39: 40.2k, Resistor_SMD:R_0805_2012Metric, F.Cu at (246.9, 129.9)
- added R40: 301k, Resistor_SMD:R_0805_2012Metric, F.Cu at (246.9, 132.8)
- added R41: 1M, Resistor_SMD:R_0805_2012Metric, F.Cu at (246.9, 135.8)
- added R42: 2.2k, Resistor_SMD:R_0805_2012Metric, F.Cu at (201.0, 59.2)
- added R43: 2.2k, Resistor_SMD:R_0805_2012Metric, F.Cu at (201.0, 62.1)
- added R44: 5.1k, Resistor_SMD:R_0805_2012Metric, F.Cu at (201.0, 65.1)
- added R45: 5.1k, Resistor_SMD:R_0805_2012Metric, F.Cu at (201.0, 68.0)
- added R46: 5.1k, Resistor_SMD:R_0805_2012Metric, F.Cu at (201.0, 71.0)
- added R47: 5.1k, Resistor_SMD:R_0805_2012Metric, F.Cu at (201.0, 74.0)
- added R48: 1M, Resistor_SMD:R_0805_2012Metric, F.Cu at (201.0, 76.9)
- added R49: 1M, Resistor_SMD:R_0805_2012Metric, F.Cu at (201.0, 79.8)
- added R50: 10k, Resistor_SMD:R_0805_2012Metric, F.Cu at (205.4, 59.2)
- added R51: 10k, Resistor_SMD:R_0805_2012Metric, F.Cu at (205.4, 62.1)
- added R52: 10k, Resistor_SMD:R_0805_2012Metric, F.Cu at (205.4, 65.1)
- added R53: 10k, Resistor_SMD:R_0805_2012Metric, F.Cu at (205.4, 68.0)
- added R54: 47, Resistor_SMD:R_0805_2012Metric, F.Cu at (205.4, 71.0)
- added R55: 1k, Resistor_SMD:R_0805_2012Metric, F.Cu at (205.4, 74.0)
- added R56: 47, Resistor_SMD:R_0805_2012Metric, F.Cu at (205.4, 76.9)
- added R57: 1k, Resistor_SMD:R_0805_2012Metric, F.Cu at (205.4, 79.8)
- added R58: 2.2k, Resistor_SMD:R_0805_2012Metric, F.Cu at (209.9, 59.2)
- added R59: 2.2k, Resistor_SMD:R_0805_2012Metric, F.Cu at (209.9, 62.1)
- added R60: 2.2k, Resistor_SMD:R_0805_2012Metric, F.Cu at (209.9, 65.1)
- added R61: 2.2k, Resistor_SMD:R_0805_2012Metric, F.Cu at (209.9, 68.0)
- added R62: 2.2k, Resistor_SMD:R_0805_2012Metric, F.Cu at (209.9, 71.0)
- added R63: 2.2k, Resistor_SMD:R_0805_2012Metric, F.Cu at (209.9, 74.0)
- added R64: 1.1k, Resistor_SMD:R_0805_2012Metric, F.Cu at (209.9, 76.9)
- added R65: 1.1k, Resistor_SMD:R_0805_2012Metric, F.Cu at (209.9, 79.8)
- added R66: 1M, Resistor_SMD:R_0805_2012Metric, F.Cu at (214.3, 59.2)
- added R67: 1M, Resistor_SMD:R_0805_2012Metric, F.Cu at (214.3, 62.1)
- added R68: 1k, Resistor_SMD:R_0805_2012Metric, F.Cu at (214.3, 65.1)
- added R69: 1k, Resistor_SMD:R_0805_2012Metric, F.Cu at (214.3, 68.0)
- added R70: 2.2k, Resistor_SMD:R_0805_2012Metric, F.Cu at (214.3, 71.0)
- added R71: 2.2k, Resistor_SMD:R_0805_2012Metric, F.Cu at (214.3, 74.0)
- added R72: 2.2k, Resistor_SMD:R_0805_2012Metric, F.Cu at (214.3, 76.9)
- added R73: 2.2k, Resistor_SMD:R_0805_2012Metric, F.Cu at (214.3, 79.8)
- added R74: 5.1k, Resistor_SMD:R_0805_2012Metric, F.Cu at (218.7, 59.2)
- added R75: 5.1k, Resistor_SMD:R_0805_2012Metric, F.Cu at (218.7, 62.1)
- added R76: 5.1k, Resistor_SMD:R_0805_2012Metric, F.Cu at (218.7, 65.1)
- added R77: 5.1k, Resistor_SMD:R_0805_2012Metric, F.Cu at (218.7, 68.0)
- added R78: 10k, Resistor_SMD:R_0805_2012Metric, F.Cu at (218.7, 71.0)
- added R79: 10k, Resistor_SMD:R_0805_2012Metric, F.Cu at (218.7, 74.0)
- added R80: 10k, Resistor_SMD:R_0805_2012Metric, F.Cu at (218.7, 76.9)
- added R81: 10k, Resistor_SMD:R_0805_2012Metric, F.Cu at (218.7, 79.8)
- added R82: 47, Resistor_SMD:R_0805_2012Metric, F.Cu at (223.1, 59.2)
- added R83: 47, Resistor_SMD:R_0805_2012Metric, F.Cu at (223.1, 62.1)
- added R84: 2.2k, Resistor_SMD:R_0805_2012Metric, F.Cu at (223.1, 65.1)
- added R85: 2.2k, Resistor_SMD:R_0805_2012Metric, F.Cu at (223.1, 68.0)
- added R86: 2.2k, Resistor_SMD:R_0805_2012Metric, F.Cu at (223.1, 71.0)
- added R87: 2.2k, Resistor_SMD:R_0805_2012Metric, F.Cu at (223.1, 74.0)
- added R88: 1.1k, Resistor_SMD:R_0805_2012Metric, F.Cu at (223.1, 76.9)
- added R89: 1.1k, Resistor_SMD:R_0805_2012Metric, F.Cu at (223.1, 79.8)
- added SW1: SW_Push, Button_Switch_THT:SW_PUSH_1P1T_6x3.5mm_H5.0_APEM_MJTP1250, F.Cu at (234.3, 83.8)
- added SW2: SW_Push, Button_Switch_THT:SW_PUSH_1P1T_6x3.5mm_H5.0_APEM_MJTP1250, F.Cu at (234.3, 88.9)
- added SW3: SW_Push, Button_Switch_THT:SW_PUSH_1P1T_6x3.5mm_H5.0_APEM_MJTP1250, F.Cu at (234.3, 94.0)
- added SW4: SW_Push, Button_Switch_THT:SW_PUSH_1P1T_6x3.5mm_H5.0_APEM_MJTP1250, F.Cu at (234.3, 99.0)
- added U10: OPA2134, Package_SO:SOIC-8_3.9x4.9mm_P1.27mm, F.Cu at (256.7, 79.1)
- added U11: TPA6110A2DGN, Package_SO:HVSSOP-8-1EP_3x3mm_P0.65mm_EP1.57x1.89mm, F.Cu at (88.3, 140.5)
- added U12: XU316-1024-TQ128-I24, SamacSys_Parts:TQFP128_196X196_XMO, F.Cu at (254.1, 104.2)
- added U13: Si5351A-B-GT, Package_SO:MSOP-10_3x3mm_P0.5mm, F.Cu at (258.9, 115.9)
- added U14: W25Q64JVSSIQ (FLASH MEMORY), SamacSys_Parts:SOIC-8_5P28X5P28_WIN, F.Cu at (250.0, 117.0)
- added U15: OPA2134, SamacSys_Parts:SOIC127P600X175-8N, F.Cu at (165.2, 135.8)
- added U16: SSM2019BRNZ, SamacSys_Parts:SOIC127P600X175-8N, F.Cu at (194.9, 60.9)
- added U17: SSM2019BRNZ, SamacSys_Parts:SOIC127P600X175-8N, F.Cu at (194.9, 67.1)
- added U18: OPA2134, SamacSys_Parts:SOIC127P600X175-8N, F.Cu at (165.2, 142.0)
- added U19: SSM2019BRNZ, SamacSys_Parts:SOIC127P600X175-8N, F.Cu at (194.9, 73.4)
- added U20: SSM2019BRNZ, SamacSys_Parts:SOIC127P600X175-8N, F.Cu at (194.9, 79.6)
- added U6: TPS82140, Package_LGA:Texas_SIL0008D_MicroSiP-8-1EP_2.8x3mm_P0.65mm_EP1.1x1.9mm_ThermalVias, F.Cu at (193.2, 125.3)
- added U9: PCM1780, Package_SO:SSOP-16_3.9x4.9mm_P0.635mm, F.Cu at (256.4, 86.0)
- added X1: FA-238 24.0000MB-C0 (CRYSTAL), SamacSys_Parts:FA-238_EPS, F.Cu at (266.5, 116.4)
- C10: value 10uF -> 120pF; footprint Capacitor_SMD:C_0805_2012Metric -> Capacitor_SMD:C_0402_1005Metric
- C11, C12, C14, C18: value 1uF -> 10uF
- C13, C17: value 1uF -> 0.1uF
- C15: value 0.1uF -> 10uF
- C19, C20: footprint Capacitor_SMD:CP_Elec_4x5.8 -> Capacitor_SMD:C_0805_2012Metric
- C2: value 4.7uF -> 120pF; footprint Capacitor_SMD:C_0805_2012Metric -> Capacitor_SMD:C_0402_1005Metric
- C21: value 0.1uF -> 2.2uF
- C22: value 10uF -> 2.2uF; footprint Capacitor_SMD:CP_Elec_4x5.8 -> Capacitor_SMD:C_0805_2012Metric
- C23: value 10uF -> 1uF; footprint Capacitor_SMD:CP_Elec_4x5.8 -> Capacitor_SMD:C_0805_2012Metric
- C24: value 1200pF -> 1uF; footprint Capacitor_SMD:C_0402_1005Metric -> Capacitor_SMD:C_0805_2012Metric
- C25: value 1200pF -> 4.7uF; footprint Capacitor_SMD:C_0402_1005Metric -> Capacitor_SMD:C_0805_2012Metric
- C26: value 120pF -> 2.2uF; footprint Capacitor_SMD:C_0402_1005Metric -> Capacitor_SMD:C_0805_2012Metric
- C27: value 120pF -> 10uF; footprint Capacitor_SMD:C_0402_1005Metric -> Capacitor_SMD:C_0805_2012Metric
- C28: value 1200pF -> 10uF; footprint Capacitor_SMD:C_0402_1005Metric -> Capacitor_SMD:C_0805_2012Metric
- C3: value 120pF -> 4.7uF; footprint Capacitor_SMD:C_0402_1005Metric -> Capacitor_SMD:C_0805_2012Metric
- C30, C31: value 120pF -> 1200pF
- C32: value 10uF -> 1200pF; footprint Capacitor_SMD:CP_Elec_4x5.8 -> Capacitor_SMD:C_0402_1005Metric
- C33, C34, C35: value 10uF -> 120pF; footprint Capacitor_SMD:CP_Elec_4x5.8 -> Capacitor_SMD:C_0402_1005Metric
- C5: value 4.7uF -> 22uF
- C6: value 120pF -> 10uF; footprint Capacitor_SMD:C_0402_1005Metric -> Capacitor_SMD:CP_Elec_4x5.8
- C8: value 22uF -> 10uF; footprint Capacitor_SMD:C_0805_2012Metric -> Capacitor_SMD:CP_Elec_4x5.8
- C9: value 1uF -> 4.7uF
- Cout5: value 22uF -> 47uF
- Cout6: value 47uF -> 22uF
- R1: value 453k -> 20k
- R10: value 20k -> 523k
- R11: value 82k -> 100k
- R12: value 20k -> 10k
- R13: value 82k -> 49.9k
- R14: value 20k -> 100k
- R15: value 82k -> 249k; footprint Resistor_SMD:R_0805_2012Metric -> Resistor_SMD:R_0603_1608Metric
- R16: value 100 -> 499k; footprint Resistor_SMD:R_0805_2012Metric -> Resistor_SMD:R_0603_1608Metric
- R17, R18: value 100 -> 8.2k
- R2: value 100k -> 52.3k
- R20: value 8.2k -> 100
- R21: value 1k -> 100
- R22: value 15k -> 100
- R23: value 100 -> 1k
- R24: value 8.2k -> 1k
- R25: value 1k -> 15k
- R3: value 200k -> 30.1k
- R4: value 100k -> 453k
- R5: value 523k -> 100k
- R6: value 100k -> 28k
- R7: value 49.9k -> 56.2k
- R8: value 100k -> 200k
- R9: value 10k -> 100k
- U2, U4: value TPS62822DLC -> TPS73601DBV; footprint Package_SON:Texas_VSON-HR-8_1.5x2mm_P0.5mm -> Package_TO_SOT_SMD:SOT-23-5
- U3: value TPS82140 -> TPS62822DLC; footprint Package_LGA:Texas_SIL0008D_MicroSiP-8-1EP_2.8x3mm_P0.65mm_EP1.1x1.9mm_ThermalVias -> Package_SON:Texas_VSON-HR-8_1.5x2mm_P0.5mm
- U5: value TPA6110A2DGN -> NCP1117-5.0_SOT223; footprint Package_SO:HVSSOP-8-1EP_3x3mm_P0.65mm_EP1.57x1.89mm -> Package_TO_SOT_SMD:SOT-223-3_TabPin2
- U7: value PCM1780 -> TPS62822DLC; footprint Package_SO:SSOP-16_3.9x4.9mm_P0.635mm -> Package_SON:Texas_VSON-HR-8_1.5x2mm_P0.5mm
- U8: value OPA2134 -> LM27761; footprint Package_SO:SOIC-8_3.9x4.9mm_P1.27mm -> Package_SON:WSON-8-1EP_2x2mm_P0.5mm_EP0.9x1.6mm
- moved U1 181.1 mm to (147.3, 123.2)
- moved U2 181.1 mm to (141.2, 123.2)
- moved U3 181.1 mm to (141.5, 117.1)
- moved J2 139.4 mm to (264.0, 17.5)
- moved J1 136.0 mm to (248.3, 17.6)
- moved U5 7.12 mm to (91.0, 78.0)
Connections:
- C1 pad 2: LEFT_IN -> AGND
- C10 pad 1: 5V -> 0.9V
- C10 pad 2: LEFT_IN -> /0.9V Power Supply/V_FB
- C11 pad 1: Net-(U5-BYPASS) -> AGND
- C11 pad 2: LEFT_IN -> AGND
- C12 pad 1: LEFT_IN -> 3.3V_LDO
- C12 pad 2: Net-(C12-Pad2) -> Net-(IC1-AVDD)
- C13 pad 1: LEFT_IN -> AGND
- C13 pad 2: Net-(C13-Pad2) -> AGND
- C14 pad 1: Net-(U6-FILT+) -> AGND
- C14 pad 2: LEFT_IN -> Net-(IC1-AVDD)
- C15 pad 1: Net-(U6-FILT+) -> Net-(IC1-AVDD)
- C15 pad 2: LEFT_IN -> AGND
- C16 pad 1: Net-(U6-VA) -> AGND
- C16 pad 2: LEFT_IN -> Net-(IC1-AVDD)
- C17 pad 1: Net-(U6-CMOUT) -> Net-(IC1-AVDD)
- C17 pad 2: LEFT_IN -> AGND
- C18 pad 1: Net-(U6-VA) -> DGND
- C18 pad 2: LEFT_IN -> 5V
- C19 pad 1: Net-(U7-V_{COM}) -> AIN_2
- C19 pad 2: LEFT_IN -> Net-(IC1-VINL2/VIN1M)
- C2 pad 1: 5V -> 3.3V
- C2 pad 2: LEFT_IN -> /3.3V Power Supply/V_FB
- C20 pad 1: 5V -> AIN_1
- C20 pad 2: LEFT_IN -> Net-(IC1-VINL1/VIN1P)
- C21 pad 1: 5V -> AGND
- C21 pad 2: LEFT_IN -> Net-(IC1-VREF)
- C22 pad 1: Net-(U7-V_{OUT}L) -> AGND
- C22 pad 2: VOUT_L -> Net-(IC1-LDO)
- C23 pad 1: Net-(U7-V_{OUT}R) -> DGND
- C23 pad 2: VOUT_R -> 5V
- C24 pad 1: Net-(C24-Pad1) -> Net-(U8-C-)
- C24 pad 2: LEFT_IN -> Net-(U8-C+)
- C25 pad 1: Net-(C24-Pad1) -> DGND
- C25 pad 2: LEFT_IN -> Net-(U8-CPOUT)
- C26 pad 1: Net-(U8A-+) -> DGND
- C26 pad 2: Net-(C26-Pad2) -> -5V
- C27 pad 1: Net-(U8A-+) -> Net-(IC1-VINL3/VIN4P)
- C27 pad 2: Net-(C26-Pad2) -> AIN_3
- C28 pad 1: Net-(C28-Pad1) -> Net-(IC1-VINL4/VIN4M)
- C28 pad 2: LEFT_IN -> AIN_4
- C29 pad 1: Net-(C28-Pad1) -> Net-(C29-Pad1)
- C29 pad 2: LEFT_IN -> AGND
- C3 pad 1: 3.3V -> 5V
- C3 pad 2: /3.3V Power Supply/V_FB -> AGND
- C30 pad 1: Net-(U8B-+) -> Net-(C30-Pad1)
- C30 pad 2: Net-(C30-Pad2) -> AGND
- C31 pad 1: Net-(U8B-+) -> Net-(C29-Pad1)
- C31 pad 2: Net-(C30-Pad2) -> AGND
- C32 pad 1: Net-(U9-CAP+) -> Net-(C30-Pad1)
- C32 pad 2: Net-(U9-CAP-) -> AGND
- C33 pad 1: LEFT_IN -> Net-(U10A--)
- C33 pad 2: -5V -> Net-(C33-Pad2)
- C34 pad 1: LEFT_IN -> Net-(U10A--)
- C34 pad 2: -5V -> Net-(C33-Pad2)
- C35 pad 1: 5V -> Net-(U10B--)
- C35 pad 2: LEFT_IN -> Net-(C35-Pad2)
- C5 pad 1: 5V -> 15V
- C5 pad 2: LEFT_IN -> AGND
- C6 pad 1: 1.8V -> 15V
- C6 pad 2: /0.9V Power Supply/V_FB -> AGND
- C7 pad 1: Net-(U3-SS/TR) -> Net-(U6-SS/TR)
- C7 pad 2: LEFT_IN -> AGND
- C8 pad 1: 15V -> 5V_LDO
- C8 pad 2: LEFT_IN -> AGND
- C9 pad 2: LEFT_IN -> AGND
- Cout1 pad 2: LEFT_IN -> AGND
- Cout2 pad 2: LEFT_IN -> AGND
- Cout3 pad 2: LEFT_IN -> AGND
- Cout4 pad 2: LEFT_IN -> AGND
- Cout5 pad 1: 1.8V -> 5V
- Cout5 pad 2: LEFT_IN -> AGND
- Cout6 pad 1: 5V -> 0.9V
- Cout6 pad 2: LEFT_IN -> AGND
- J1 pad R: LEFT_IN -> RIGHT_IN
- J1 pad S: LEFT_IN -> AGND
- J2 pad S: LEFT_IN -> AGND
- L3 pad 2: 1.8V -> 0.9V
- R1 pad 1: 3.3V -> 5V
- R1 pad 2: /3.3V Power Supply/V_FB -> Net-(U1-EN)
- R10 pad 2: Net-(U1-EN) -> /5V Power Supply/V_FB
- R11 pad 1: Net-(U5-SHDN) -> /5V Power Supply/V_FB
- R11 pad 2: LEFT_IN -> AGND
- R12 pad 1: Net-(C12-Pad2) -> 5V
- R12 pad 2: Net-(U5-IN1-) -> 0.9V_EN
- R13 pad 1: LEFT_OUT -> 0.9V
- R13 pad 2: Net-(U5-IN1-) -> /0.9V Power Supply/V_FB
- R14 pad 1: Net-(C13-Pad2) -> /0.9V Power Supply/V_FB
- R14 pad 2: Net-(U5-IN2-) -> AGND
- R15 pad 1: Net-(U5-IN2-) -> -5V
- R15 pad 2: RIGHT_OUT -> Net-(U8-VFB)
- R16 pad 1: MCLK -> Net-(U8-VFB)
- R16 pad 2: Net-(U7-SCK) -> DGND
- R17 pad 1: DATA_LR_CLOCK -> VOUT_L
- R17 pad 2: Net-(U7-LRCK) -> Net-(C29-Pad1)
- R18 pad 1: DATA -> VOUT_R
- R18 pad 2: Net-(U7-DATA) -> Net-(C30-Pad1)
- R19 pad 1: DATA_BIT_CLOCK -> BCK
- R19 pad 2: Net-(U7-BCK) -> Net-(U9-BCK)
- R2 pad 1: /3.3V Power Supply/V_FB -> 3.3V_LDO
- R2 pad 2: LEFT_IN -> Net-(U2-FB)
- R20 pad 1: VOUT_L -> MCLK
- R20 pad 2: Net-(C24-Pad1) -> Net-(U9-SCK)
- R21 pad 1: Net-(C24-Pad1) -> LRCK
- R21 pad 2: Net-(U8A-+) -> Net-(U9-LRCK)
- R22 pad 1: Net-(C24-Pad1) -> DATA
- R22 pad 2: Net-(C26-Pad2) -> Net-(U9-DATA)
- R23 pad 1: Net-(C26-Pad2) -> Net-(C29-Pad1)
- R23 pad 2: LEFT_IN -> Net-(U10A--)
- R24 pad 1: VOUT_R -> Net-(C30-Pad1)
- R24 pad 2: Net-(C28-Pad1) -> Net-(U10B--)
- R25 pad 1: Net-(C28-Pad1) -> Net-(C29-Pad1)
- R25 pad 2: Net-(U8B-+) -> Net-(C33-Pad2)
- R26 pad 1: Net-(C28-Pad1) -> Net-(C30-Pad1)
- R26 pad 2: Net-(C30-Pad2) -> Net-(C35-Pad2)
- R27 pad 1: Net-(C30-Pad2) -> Net-(C33-Pad2)
- R3 pad 1: 1.8V -> Net-(U2-FB)
- R3 pad 2: /1.8V Power Supply/V_FB -> AGND
- R4 pad 1: /1.8V Power Supply/V_FB -> 3.3V
- R4 pad 2: LEFT_IN -> /3.3V Power Supply/V_FB
- R5 pad 1: 5V -> /3.3V Power Supply/V_FB
- R5 pad 2: /5V Power Supply/V_FB -> AGND
- R6 pad 1: /5V Power Supply/V_FB -> 1.8V_LDO
- R6 pad 2: LEFT_IN -> Net-(U4-FB)
- R7 pad 1: 1.8V -> Net-(U4-FB)
- R7 pad 2: /0.9V Power Supply/V_FB -> AGND
- R8 pad 1: /0.9V Power Supply/V_FB -> 1.8V
- R8 pad 2: LEFT_IN -> /1.8V Power Supply/V_FB
- R9 pad 1: 5V -> /1.8V Power Supply/V_FB
- R9 pad 2: 0.9V_EN -> AGND
- Rpg1 pad 2: Net-(U2-PG) -> 0.9V_EN
- Rpg2 pad 2: 0.9V_EN -> Net-(U3-PG)
- Rpg3 pad 1: 5V -> Net-(U6-PG)
- Rpg3 pad 2: Net-(U4-PG) -> 5V
- Rpg4 pad 1: Net-(U3-PG) -> 5V
- Rpg4 pad 2: 5V -> Net-(U7-PG)
- U1 pad 3: LEFT_IN -> AGND
- U1 pad 5: LEFT_IN -> AGND
- U2 pad 2: /1.8V Power Supply/V_FB -> AGND
- U2 pad 3: LEFT_IN -> 5V
- U2 pad 4: unconnected-(U2-NC-Pad4) -> Net-(U2-FB)
- U2 pad 5: LEFT_IN -> 3.3V_LDO
- U3 pad 1: 15V -> 5V
- U3 pad 2: 15V -> /1.8V Power Supply/V_FB
- U3 pad 3: LEFT_IN -> AGND
- U3 pad 4: 5V -> unconnected-(U3-NC-Pad4)
- U3 pad 5: 5V -> AGND
- U3 pad 6: /5V Power Supply/V_FB -> /1.8V Power Supply/V_Buck
- U3 pad 7: Net-(U3-PG) -> 5V
- U3 pad 8: Net-(U3-SS/TR) -> Net-(U3-PG)
- U4 pad 1: 0.9V_EN -> 5V
- U4 pad 2: /0.9V Power Supply/V_FB -> AGND
- U4 pad 3: LEFT_IN -> 5V
- U4 pad 4: unconnected-(U4-NC-Pad4) -> Net-(U4-FB)
- U4 pad 5: LEFT_IN -> 1.8V_LDO
- U5 pad 1: Net-(U5-BYPASS) -> AGND
- U5 pad 2: LEFT_IN -> 5V_LDO
- U5 pad 3: Net-(U5-SHDN) -> 15V
- U7 pad 1: ZERO_L -> 0.9V_EN
- U7 pad 2: MODE_CONTROL_SELECT -> /0.9V Power Supply/V_FB
- U7 pad 3: MODE_CONTROL_CLOCK -> AGND
- U7 pad 4: MODE_CONTROL_DATA -> unconnected-(U7-NC-Pad4)
- U7 pad 5: Net-(U7-SCK) -> AGND
- U7 pad 6: Net-(U7-DATA) -> /0.9V Power Supply/V_Buck
- U7 pad 7: Net-(U7-BCK) -> 5V
- U7 pad 8: Net-(U7-LRCK) -> Net-(U7-PG)
- U8 pad 1: Net-(C26-Pad2) -> 5V
- U8 pad 2: LEFT_IN -> DGND
- U8 pad 3: Net-(U8A-+) -> Net-(U8-CPOUT)
- U8 pad 5: Net-(U8B-+) -> Net-(U8-VFB)
- U8 pad 6: LEFT_IN -> 5V
- U8 pad 7: Net-(C30-Pad2) -> Net-(U8-C-)
- U8 pad 8: 5V -> Net-(U8-C+)
Other:
- copper layers 2 -> 4

Commit message: Added BIG KNOB schematic and started PCB
Parts:
- added C202: 100nF, Capacitor_SMD:C_0402_1005Metric, F.Cu at (55.1, 140.0)
- added C203: 100nF, Capacitor_SMD:C_0402_1005Metric, F.Cu at (55.1, 141.9)
- added C204: 100nF, Capacitor_SMD:C_0402_1005Metric, F.Cu at (55.1, 143.9)
- added C205: 100nF, Capacitor_SMD:C_0402_1005Metric, F.Cu at (55.1, 145.9)
- added C206: 2.2uF, Capacitor_SMD:C_0402_1005Metric, F.Cu at (55.1, 147.8)
- added C207: 100nF, Capacitor_SMD:C_0402_1005Metric, F.Cu at (55.1, 149.8)
- added C208: 100nF, Capacitor_SMD:C_0402_1005Metric, F.Cu at (55.1, 151.8)
- added C209: 100nF, Capacitor_SMD:C_0402_1005Metric, F.Cu at (58.0, 140.0)
- added C210: 100nF, Capacitor_SMD:C_0402_1005Metric, F.Cu at (58.0, 141.9)
- added C211: 100nF, Capacitor_SMD:C_0402_1005Metric, F.Cu at (58.0, 143.9)
- added C212: 100nF, Capacitor_SMD:C_0402_1005Metric, F.Cu at (58.0, 145.9)
- added C213: 100nF, Capacitor_SMD:C_0402_1005Metric, F.Cu at (58.0, 147.8)
- added C214: 100nF, Capacitor_SMD:C_0402_1005Metric, F.Cu at (58.0, 149.8)
- added C215: 100nF, Capacitor_SMD:C_0402_1005Metric, F.Cu at (58.0, 151.8)
- added C216: 100nF, Capacitor_SMD:C_0402_1005Metric, F.Cu at (60.9, 140.0)
- added C217: 100nF, Capacitor_SMD:C_0402_1005Metric, F.Cu at (60.9, 141.9)
- added C218: 100nF, Capacitor_SMD:C_0402_1005Metric, F.Cu at (60.9, 143.9)
- added C219: 10uF, Capacitor_SMD:C_0805_2012Metric, F.Cu at (124.0, 103.9)
- added C220: 10uF, Capacitor_SMD:C_0805_2012Metric, F.Cu at (128.9, 103.2)
- added C221: 0.1uF, Capacitor_SMD:C_0805_2012Metric, F.Cu at (121.5, 103.9)
- added C222: 10uF, Capacitor_SMD:C_0805_2012Metric, F.Cu at (136.3, 106.2)
- added C223: 10uF, Capacitor_SMD:C_0805_2012Metric, F.Cu at (132.9, 106.3)
- added C224: 0.1uF, Capacitor_SMD:C_0805_2012Metric, F.Cu at (138.6, 106.2)
- added C225: 0.1uF, Capacitor_SMD:C_0805_2012Metric, F.Cu at (130.6, 106.2)
- added C226: 10uF, Capacitor_SMD:C_0805_2012Metric, F.Cu at (124.9, 94.3)
- added C227: 10uF, Capacitor_SMD:C_0805_2012Metric, F.Cu at (124.8, 96.3)
- added C228: 2.2uF, Capacitor_SMD:C_0805_2012Metric, F.Cu at (129.8, 98.6)
- added C229: 2.2uF, Capacitor_SMD:C_0805_2012Metric, F.Cu at (125.8, 100.8)
- added C230: 10uF, Capacitor_SMD:C_0805_2012Metric, F.Cu at (144.8, 95.0)
- added C231: 10uF, Capacitor_SMD:C_0805_2012Metric, F.Cu at (144.9, 97.3)
- added C232: 1uF, Capacitor_SMD:C_0402_1005Metric, F.Cu at (60.9, 145.9)
- added C234: 0.01uF, Capacitor_SMD:C_0402_1005Metric, F.Cu at (158.3, 125.3)
- added C235: 0.01uF, Capacitor_SMD:C_0402_1005Metric, F.Cu at (158.3, 131.4)
- added IC5: PCM1865DBT, SamacSys_Parts:SOP50P640X120-30N, F.Cu at (135.6, 98.9)
- added J21: Line Out (Right), Connector_Audio:Jack_3.5mm_CUI_SJ-3523-SMT_Horizontal, F.Cu at (249.1, 18.0)
- added R164: 0, Resistor_SMD:R_0805_2012Metric, F.Cu at (64.5, 140.4)
- added R165: 43, Resistor_SMD:R_0805_2012Metric, F.Cu at (64.5, 143.4)
- added R166: 43, Resistor_SMD:R_0805_2012Metric, F.Cu at (64.5, 146.3)
- added R167: 3k, Resistor_SMD:R_0805_2012Metric, F.Cu at (149.4, 176.1)
- added R168: 3k, Resistor_SMD:R_0805_2012Metric, F.Cu at (152.0, 176.1)
- added R169: 3k, Resistor_SMD:R_0805_2012Metric, F.Cu at (149.2, 185.8)
- added R170: 3k, Resistor_SMD:R_0805_2012Metric, F.Cu at (152.1, 185.8)
- added R175: 10k, Resistor_SMD:R_0805_2012Metric, F.Cu at (151.2, 127.7)
- added R176: 10k, Resistor_SMD:R_0805_2012Metric, F.Cu at (151.2, 130.3)
- added R177: 10k, Resistor_SMD:R_0805_2012Metric, F.Cu at (154.8, 127.7)
- added R178: 10k, Resistor_SMD:R_0805_2012Metric, F.Cu at (154.9, 130.3)
- added U34: NE5532AD, PCM_Package_SO_AKL:SO-8_3.9x4.9mm_P1.27mm, F.Cu at (157.4, 187.3)
- added U35: NE5532AD, PCM_Package_SO_AKL:SO-8_3.9x4.9mm_P1.27mm, F.Cu at (157.1, 177.4)
- added X2: FA-238 24.0000MB-C0, SamacSys_Parts:FA-238_EPS, F.Cu at (66.2, 150.7)
- IC2: footprint SamacSys_Parts:SOP65P490X110-9N -> SamacSys_Parts:SOP50P490X110-11N
- J1: value Line Out -> Line Out (Left)
- R12, R13, R14, Rpg4: footprint Resistor_SMD:R_0805_2012Metric -> PCM_Resistor_SMD_AKL:R_0805_2012Metric_Pad1.15x1.40mm_HandSolder
- moved U9 230.6 mm to (46.3, 180.9)
- moved C37 226.6 mm to (62.7, 179.6)
- moved C38 223.1 mm to (62.2, 183.2)
- moved C40 220.1 mm to (62.0, 189.1)
- moved C43 219.9 mm to (51.5, 187.4), turned to -90 degrees
- moved C39 216.1 mm to (62.0, 175.5)
- moved R28 207.0 mm to (93.3, 183.1)
- moved U10 202.2 mm to (83.6, 183.6)
- moved C36 197.5 mm to (89.3, 184.1)
- moved C42 196.2 mm to (83.3, 189.8), turned to 180 degrees
- moved C41 181.8 mm to (96.1, 177.1)
- moved L4 153.5 mm to (98.3, 144.6), turned to -90 degrees
- moved C52 149.9 mm to (101.5, 145.6), turned to 90 degrees
- moved C51 149.2 mm to (102.2, 143.4), turned to 180 degrees
- moved IC2 148.7 mm to (105.5, 145.9)
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Connections:
- net Net-(U12A-XIN) renamed XIN
- net Net-(U12A-XOUT) renamed XOUT
- IC1 pad 15: SCKI -> MCLK
- J1 pad R: RIGHT_IN -> LEFT_OUT+
- J1 pad T: LEFT_IN -> LEFT_OUT-
- J20 pad 1: Net-(C58-Pad2) -> AGND
- J20 pad 3: AGND -> Net-(C58-Pad2)
- J5 pad 1: Net-(C59-Pad2) -> AGND
- J5 pad 3: AGND -> Net-(C59-Pad2)
- J6 pad 1: Net-(C81-Pad2) -> AGND
- J6 pad 3: LEFT_IN -> Net-(C81-Pad2)
- J7 pad 1: Net-(C80-Pad2) -> AGND
- J7 pad 3: LEFT_IN -> Net-(C80-Pad2)
- U12 pad 10: unconnected-(U12A-VDDIOL-Pad10) -> 1.8V_LDO
- U12 pad 104: unconnected-(U12B-VDD-Pad104) -> 0.9V
- U12 pad 105: unconnected-(U12B-VDD-Pad105) -> 0.9V
- U12 pad 106: unconnected-(U12B-VDD-Pad106) -> 0.9V
- U12 pad 109: unconnected-(U12B-VDDIOT-Pad109) -> 1.8V_LDO
- U12 pad 11: unconnected-(U12A-VDD-Pad11) -> 0.9V
- U12 pad 113: unconnected-(U12B-VDD-Pad113) -> 0.9V
- U12 pad 121: unconnected-(U12B-VDDIOT-Pad121) -> 1.8V_LDO
- U12 pad 129: unconnected-(U12B-GND-Pad129) -> AGND
- U12 pad 14: unconnected-(U12A-VDD-Pad14) -> 0.9V
- U12 pad 17: unconnected-(U12A-VDDIOL-Pad17) -> 1.8V_LDO
- U12 pad 18: unconnected-(U12A-VDD-Pad18) -> 0.9V
- U12 pad 24: unconnected-(U12A-MIPI_VDD18-Pad24) -> AGND
- U12 pad 27: unconnected-(U12A-MIPI_VDD09-Pad27) -> AGND
- U12 pad 30: unconnected-(U12A-GND-Pad30) -> AGND
- U12 pad 35: unconnected-(U12A-VDDIOB18-Pad35) -> 1.8V_LDO
- U12 pad 36: unconnected-(U12A-TDI-Pad36) -> TDI
- U12 pad 37: unconnected-(U12A-TDO-Pad37) -> TDO
- U12 pad 38: unconnected-(U12A-RST_N-Pad38) -> RST_N
- U12 pad 39: unconnected-(U12A-VDD-Pad39) -> 0.9V
- U12 pad 40: unconnected-(U12A-LV_L_N-Pad40) -> AGND
- U12 pad 41: unconnected-(U12A-PLL_AVDD-Pad41) -> Net-(U12A-PLL_AVDD)
- U12 pad 42: unconnected-(U12A-PLL_AGND-Pad42) -> AGND
- U12 pad 43: unconnected-(U12A-LV_T_N-Pad43) -> AGND
- U12 pad 44: unconnected-(U12A-TMS-Pad44) -> TMS
- U12 pad 45: unconnected-(U12A-VDD-Pad45) -> 0.9V
- U12 pad 5: unconnected-(U12A-VDD-Pad5) -> 0.9V
- U12 pad 50: unconnected-(U12A-VDD-Pad50) -> 0.9V
- U12 pad 51: unconnected-(U12A-TCK-Pad51) -> TCK
- U12 pad 52: unconnected-(U12A-LV_R_N-Pad52) -> AGND
- U12 pad 54: unconnected-(U12A-VDD-Pad54) -> 0.9V
- U12 pad 56: unconnected-(U12A-VDDIOB18-Pad56) -> 1.8V_LDO
- U12 pad 59: unconnected-(U12A-USB_DM-Pad59) -> USB_DN
- U12 pad 60: unconnected-(U12A-USB_DP-Pad60) -> USB_DP
- U12 pad 61: unconnected-(U12A-USB_VDD33-Pad61) -> 3.3V_LDO
- U12 pad 62: unconnected-(U12A-USB_VDD18-Pad62) -> 1.8V_LDO
- U12 pad 66: unconnected-(U12B-X1D16-Pad66) -> XL_DN1
- U12 pad 67: unconnected-(U12B-X1D17-Pad67) -> XL_DN0
- U12 pad 68: unconnected-(U12B-VDD-Pad68) -> 0.9V
- U12 pad 69: unconnected-(U12B-X1D18-Pad69) -> XL_UP0
- U12 pad 70: unconnected-(U12B-X1D19-Pad70) -> XL_UP1
- U12 pad 72: unconnected-(U12B-VDDIOR-Pad72) -> 1.8V_LDO
- U12 pad 85: unconnected-(U12B-VDD-Pad85) -> 0.9V
- U12 pad 89: unconnected-(U12B-VDDIOR-Pad89) -> 1.8V_LDO
- U12 pad 95: unconnected-(U12B-VDD-Pad95) -> 0.9V
Other:
- board text added: "0.9V Circuitry"
- board text added: "1.8V Circuitry"
- board text added: "3.3V Circuitry"
- board text added: "36V Generator"
- board text added: "5V Circuitry"
- board text added: "DAC"
- board text added: "DAC Circuitry"
- board text added: "Headphone Amp"
- board text added: "Headphone Out"
- board text added: "Left ADC"
- board text added: "Left Out (+/-)"
- board text added: "Line Out L R"
- board text added: "Post DAC LPF"
- board text added: "Power Input Circuitry"
- board text added: "Right ADC"
- board text added: "Right Out (+/-)"
- board text added: "Rotary Encoder (Missing Footprint)"
- board text added: "Takes 15V in"
- board text added: "Takes 5V in"
- board text added: "Takes 5V in Output enables 0.9V"
- board text added: "Voltage Inverter"

Commit message: initial placement of all cmponents
need to add:
- pin headers for Rpi
- separate the boards and add pin headers for connection points
- probably get rid of buck converters and change LDOs to be higher current
Parts:
- added FL1: BLM18AG601SZ1D, SamacSys_Parts:BLM18SP221SN1B, F.Cu at (161.4, 122.0)
- added J22: 2171790001, Connector_Molex:Molex_Micro-Fit_3.0_43045-1615_2x08_P3.00mm_Vertical, F.Cu at (192.8, 153.9)
- added J8: FTSH-110-01-F-DV-K, SamacSys_Parts:FTSH-110-XX-YYY-DV-K-A, F.Cu at (186.2, 131.1)
- added U37: PEC11R-4030F-N0024, SamacSys_Parts:PEC11R4030FN0024, F.Cu at (62.9, 141.4)
- moved J10 269.2 mm to (186.3, 241.4)
- moved C79 246.0 mm to (120.4, 277.3)
- moved C75 240.4 mm to (105.0, 273.5), turned to 180 degrees
- moved C68 234.9 mm to (95.9, 255.0), turned to 90 degrees
- moved C83 231.7 mm to (127.5, 272.8), turned to 90 degrees
- moved C55 229.8 mm to (103.7, 252.1), turned to 90 degrees
- moved C61 224.6 mm to (95.5, 251.9)
- moved R52 224.3 mm to (96.0, 258.4), turned to -90 degrees
- moved R63 224.3 mm to (117.3, 276.0), turned to 90 degrees
- moved R62 223.8 mm to (117.2, 272.5), turned to -90 degrees
- moved R43 223.5 mm to (101.7, 260.0), turned to 180 degrees
- moved C69 222.3 mm to (114.2, 254.0), turned to 90 degrees
- moved U17 220.9 mm to (122.8, 274.0)
- moved C57 220.0 mm to (114.7, 251.4), turned to 180 degrees
- moved C105 218.7 mm to (189.6, 276.1)
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Other:
- board text added: "36V Generator (For Phantom Power)"
- board text added: "ADC Circuitry"
- board text added: "Combo TRS-XLR In 1"
- board text added: "Combo TRS-XLR In 2"
- board text added: "Combo TRS-XLR In 3"
- board text added: "Combo TRS-XLR In 4"
- board text added: "Crystal Circuit"
- board text added: "Flash Memory"
- board text added: "Preamps for TS 1-4"
- board text added: "Rotary Encoder (for Rpi)"
- board text added: "TS in 1/2"
- board text added: "TS in 3/4"
- board text added: "Voltage Inverter (For Dual Supply Op Amp)"
- board text added: "Xcore Crystal"
- board text added: "Xcore DSP Chip"
- board text added: "Xcore Pin Header"
- board text removed: "36V Generator"
- board text removed: "Rotary Encoder (Missing Footprint)"
- board text removed: "Voltage Inverter"
