File: Power_Supplies_DSP/XCORE.kicad_sch (KiCad schematic)
At the start: 47 parts, among them J22 USB_C_Receptacle_USB2.0, J35 PINHD_1x1_Female, J41 PINHD_1x10_Female, J8 FTSH-110-01-F-DV-K, U1 PEC11R-4030F-N0024, U12 XU316-1024-TQ128-I24, U13 Si5351A-B-GT, U14 W25Q64JVSSIQ (FLASH MEMORY), X1 FA-238 24.0000MB-C0 (CRYSTAL), X2 FA-238 24.0000MB-C0

Commit message: mcu PCB
Parts:
- C1, C2, C202, C203, C204, C205, C206, C207, C208, C209, C210, C211, C212, C213, C214, C215, C216, C217, C218, C232, C49, C50: footprint Capacitor_SMD:C_0402_1005Metric -> Capacitor_SMD:C_0603_1608Metric_Pad1.08x0.95mm_HandSolder
