File: Power_Supplies_DSP/Power_Supplies_DSP.kicad_sch (KiCad schematic)
At the start: 0 parts

Commit message: STM32 schematic started
Other:
- added sheet STM32 (stm32.kicad_sch)
Changed lines of the file:
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@@
+	)
+	(sheet
+		(at 114.3 99.06)
+		(size 38.1 19.05)
+		(fields_autoplaced yes)
+		(stroke
+			(width 0.1524)
+			(type solid)
+		)
+		(fill
+			(color 0 0 0 0.0000)
+		)
+		(property "Sheetname" "STM32"
+			(at 114.3 98.3484 0)
+			(effects
+				(font
+					(size 1.27 1.27)
+				)
+				(justify left bottom)
+			)
+		)
+		(property "Sheetfile" "stm32.kicad_sch"
+			(at 114.3 118.6946 0)
+			(effects
+				(font
+					(size 1.27 1.27)
+				)
+				(justify left top)
+			)
+		)
+		(instances
+			(project "Power_Supplies_DSP"
+				(path "/5266cf9e-da90-4c53-80fd-cf3dbed42632"
+					(page "3")
+				)
+			)
+		)
 	)
 	(sheet

Commit message: stuff i may or may not have done to order these things
Other:
- removed sheet Xcore
Changed lines of the file:
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@@
-		)
-	)
-	(sheet
-		(at 111.76 60.96)
-		(size 40.64 22.86)
-		(fields_autoplaced yes)
-		(stroke
-			(width 0.1524)
-			(type solid)
-		)
-		(fill
-			(color 0 0 0 0.0000)
-		)
-		(property "Sheetname" "Xcore"
-			(at 111.76 60.2484 0)
-			(effects
-				(font
-					(size 1.27 1.27)
-				)
-				(justify left bottom)
-			)
-		)
-		(property "Sheetfile" "XCORE.kicad_sch"
-			(at 111.76 84.4046 0)
-			(effects
-				(font
-					(size 1.27 1.27)
-				)
-				(justify left top)
-			)
-		)
-		(instances
-			(project "Power_Supplies_DSP"
-				(path "/5266cf9e-da90-4c53-80fd-cf3dbed42632"
-					(page "9")
-				)
-			)
 		)
 	)
