File: Power_Supplies_MAIN/Power_Supplies.kicad_pcb (KiCad board)
At the start: 4 copper layers, 324.8 x 181.8 mm, 228 parts, among them IC1 PCM1865DBT, IC2 LM2940IMPX-10_NOPB, IC3 XC6902NA01PR-G, IC5 PCM1865DBT, J1 Line Out (Left), J10 XLR3_AudioJack3_Combo, J11 PINHD_1x4_Female, J12 PINHD_1x8_Female, J2 Headphone Out, J20 ACJM-MV-2, J21 Line Out (Right), J29 PINHD_1x2_Female, J3 XLR3_AudioJack3_Combo, J30 PINHD_1x2_Female, J31 PINHD_1x2_Female, J32 PINHD_1x2_Female, J33 PINHD_1x3_Female, J36 PINHD_1x2_Female, J4 XLR3_AudioJack3_Combo, J5 ACJM-MV-2, J6 ACJM-MV-2, J7 ACJM-MV-2, J8 PINHD_1x3_Female, J9 XLR3_AudioJack3_Combo, U10 OPA2134, U11 TPA6110A2DGN, U15 OPA2134, U16 SSM2019BRNZ, U17 SSM2019BRNZ, U18 OPA2134, U19 SSM2019BRNZ, U20 SSM2019BRNZ, U34 NE5532AD, U35 NE5532AD, U9 PCM1780

Commit message: updated main PCB to reflect changes w/ new mcu
Parts:
- removed J12: PINHD_1x8_Female, Connector_PinSocket_2.54mm:PinSocket_1x08_P2.54mm_Vertical
- removed J8: PINHD_1x3_Female, Connector_PinSocket_2.54mm:PinSocket_1x03_P2.54mm_Vertical
- added J13: PINHD_1x10_Female, Connector_PinSocket_2.54mm:PinSocket_1x10_P2.54mm_Vertical, F.Cu at (141.2, 184.3)
- added J14: PINHD_1x10_Female, Connector_PinSocket_2.54mm:PinSocket_1x10_P2.54mm_Vertical, F.Cu at (141.2, 214.3)
- moved R180 23.3 mm to (137.3, 166.3)
- moved R43 23.3 mm to (140.1, 166.3)
Connections:
- IC1 pad 16: LRCK -> LRCK_ADC
- IC1 pad 17: BCK -> BCLK_ADC
- IC5 pad 16: LRCK -> LRCK_ADC
- IC5 pad 17: BCK -> BCLK_ADC
- R180 pad 2: DATA_OUT_1 -> DIN
- R19 pad 1: BCK -> BCLK_DAC
- R21 pad 1: LRCK -> LRCK_DAC
- R43 pad 2: DATA_OUT_2 -> DIN
Routing:
- net BCK: track 309.1 -> 0.00 mm, vias 5 -> 0
- net LRCK: track 269.6 -> 0.00 mm, vias 4 -> 0
- net LRCK_DAC: track 0.00 -> 186.6 mm, vias 0 -> 2
- net BCLK_DAC: track 0.00 -> 178.7 mm, vias 0 -> 2
- net BCLK_ADC: track 0.00 -> 122.4 mm, vias 0 -> 3
- net LRCK_ADC: track 0.00 -> 114.9 mm, vias 0 -> 6
- net 3.3V_2: track 142.1 -> 233.8 mm, vias 0 -> 4
- net 3.3V: track 252.4 -> 336.3 mm
- net AGND: track 324.8 -> 408.3 mm
- net SCL: track 115.9 -> 182.6 mm, vias 5 -> 4
- net DIN: track 0.00 -> 44.2 mm, vias 0 -> 2
- net 5V: track 270.8 -> 312.5 mm, vias 5 -> 7
- net SDA: track 119.6 -> 146.8 mm, vias 4 -> 5
- net Net-(IC1-DOUT): track 44.5 -> 20.6 mm
- net Net-(IC5-DOUT): track 104.2 -> 80.4 mm
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Other:
- board text added: "Pins to MCU"
- board text removed: "5V"
- board text removed: "DATA"
- board text removed: "DATA_OUT1"
- board text removed: "Digital Power Pins"
- board text removed: "Pins to Xcore"

Commit message: added changes that weeks wanted 🐷
Parts:
- removed C11, C12, C220: 10uF, Capacitor_SMD:C_0805_2012Metric
- added R2: 0R, Resistor_SMD:R_0805_2012Metric_Pad1.20x1.40mm_HandSolder, F.Cu at (171.2, 145.6)
- added R3: 0R, Resistor_SMD:R_0805_2012Metric_Pad1.20x1.40mm_HandSolder, F.Cu at (107.7, 145.6)
- added R4: 1k, Resistor_SMD:R_0805_2012Metric_Pad1.20x1.40mm_HandSolder, F.Cu at (130.4, 150.9)
- added R5: 1k, Resistor_SMD:R_0805_2012Metric_Pad1.20x1.40mm_HandSolder, F.Cu at (195.3, 150.5)
- R1: value 1k -> 0R
- moved R37 2.93 mm to (200.1, 152.1)
Connections:
- C14 pad 2: Net-(IC1-AVDD) -> 3.3V
- C15 pad 1: Net-(IC1-DVDD) -> 3.3V_2
- C16 pad 2: Net-(IC1-AVDD) -> 3.3V
- C17 pad 1: Net-(IC1-DVDD) -> 3.3V_2
- C222 pad 2: Net-(IC5-AVDD) -> 3.3V
- C223 pad 1: Net-(IC5-DVDD) -> 3.3V_2
- C224 pad 2: Net-(IC5-AVDD) -> 3.3V
- C225 pad 1: Net-(IC5-DVDD) -> 3.3V_2
- IC1 pad 13: Net-(IC1-DVDD) -> 3.3V_2
- IC1 pad 14: Net-(IC1-DVDD) -> 3.3V_2
- IC1 pad 15: MCLK -> Net-(IC1-SCKI)
- IC1 pad 8: Net-(IC1-AVDD) -> 3.3V
- IC5 pad 13: Net-(IC5-DVDD) -> 3.3V_2
- IC5 pad 14: Net-(IC5-DVDD) -> 3.3V_2
- IC5 pad 15: unconnected-(IC5-SCKI-Pad15) -> Net-(IC5-SCKI)
- IC5 pad 8: Net-(IC5-AVDD) -> 3.3V
- J14 pad 10: AGND -> unconnected-(J14-Pad10)
Routing:
- net AGND: track 408.3 -> 328.6 mm, vias 162 -> 164
- net MCLK: track 234.0 -> 278.0 mm, vias 4 -> 5
- net 3.3V: track 336.3 -> 369.3 mm
- net 3.3V_2: track 233.8 -> 249.6 mm
- net Net-(IC1-AVDD): track 15.1 -> 0.00 mm
- net Net-(IC5-AVDD): track 14.3 -> 0.00 mm
- net Net-(IC5-DVDD): track 13.9 -> 0.00 mm
- net DGND: track 25.3 -> 28.9 mm, vias 13 -> 15
- net Net-(IC5-MC/SCL): track 7.85 -> 11.2 mm
- net SCL: track 182.6 -> 185.7 mm
- net Net-(IC5-SCKI): track 0.00 -> 2.37 mm
- net Net-(IC1-SCKI): track 0.00 -> 1.80 mm
- added copper zone on F.Cu, net (none)
Other:
- board size 324.8 x 181.8 mm -> 343.1 x 201.9 mm
