File: Audio_Board_Analog_Only/LDO.kicad_sch (KiCad schematic)
At the start: 54 parts, among them IC1 LM2940IMPX-10_NOPB, IC10 XC6902NA01PR-G, IC2 LM2940IMPX-10_NOPB, IC4 XC6902NA01PR-G, IC5 LM2940IMPX-10_NOPB, IC6 XC6902NA01PR-G, IC7 LM2940IMPX-10_NOPB, IC8 XC6902NA01PR-G, IC9 LM2940IMPX-10_NOPB

Commit message: made new pcbs :(
Parts:
- removed C5: 0.47uF, PCM_Capacitor_SMD_AKL:C_0805_2012Metric, symbol PCM_Capacitor_AKL:C_0805
- removed C6: 22uF, Capacitor_SMD:CP_Elec_4x5.8, symbol Device:C_Polarized_US
- removed D7: LED, LED_SMD:LED_0402_1005Metric_Pad0.77x0.64mm_HandSolder, symbol PCM_SL_Devices:LED
- removed IC2: LM2940IMPX-10_NOPB, SamacSys_Parts:SOT230P700X180-4N, symbol SamacSys_Parts:LM2940IMPX-10_NOPB
- removed R11: 2.2k, Resistor_SMD:R_0805_2012Metric, symbol Device:R
- removed R21: 0, Resistor_SMD:R_0805_2012Metric, symbol Device:R
- added C1, C24, C25: 1uF, Capacitor_SMD:C_0402_1005Metric, symbol Device:C
- added C2: 0.1uF, Capacitor_SMD:C_0402_1005Metric, symbol Device:C
- added C7: 0.01uF, Capacitor_SMD:C_0402_1005Metric, symbol Device:C
- added C8: 0.001uF, Capacitor_SMD:C_0402_1005Metric, symbol Device:C
- added D8: LED, LED_SMD:LED_0402_1005Metric_Pad0.77x0.64mm_HandSolder, symbol PCM_SL_Devices:LED
- added IC3: TPS73250DBVR, SamacSys_Parts:SOT95P280X145-5N, symbol SamacSys_Parts:TPS73250DBVR
- added R22: 0, Resistor_SMD:R_0805_2012Metric, symbol Device:R
- added R34: 2.2k, Resistor_SMD:R_0805_2012Metric, symbol Device:R
- IC4: value XC6902NA01PR-G -> XC6902NA51PR-G
Connections:
- net 5V: now also R22.2
- net 5V_Filtered: now also C25.1, D8.2, IC3.5 (OUT)
- net AGND: now also C1.1, C2.1, C24.1, C25.2, C7.1, C8.1, IC3.2 (GND), R34.2
- new net: C1.2, C2.2, C7.2, C8.2, IC3.1 (IN), IC3.3 (EN), R22.1
- new net: D8.1, R34.1
- new net: C24.2, IC3.4 (NR/FB)
Other:
- note added: "-10.5V Output"
