File: Audio_Board_Analog_Only/PREAMPS.kicad_sch (KiCad schematic)
At the start: 132 parts, among them J10 XLR3_AudioJack3_Combo, J17 PINHD_1x3_Male, J18 PINHD_1x2_Male, J20 ACJM-MV-2, J3 XLR3_AudioJack3_Combo, J4 XLR3_AudioJack3_Combo, J5 ACJM-MV-2, J6 ACJM-MV-2, J7 ACJM-MV-2, J9 XLR3_AudioJack3_Combo, U15 OPA2134, U16 SSM2019BRNZ, U17 SSM2019BRNZ, U18 OPA2134, U19 SSM2019BRNZ, U20 SSM2019BRNZ

Commit message: made new pcbs :(
Parts:
- added J12: PINHD_1x2_Male, Connector_PinHeader_2.54mm:PinHeader_1x02_P2.54mm_Vertical, symbol PCM_SL_Pin_Headers:PINHD_1x2_Male
Connections:
- net AGND: now also J12.1
- net AIN_8: now also J12.2
Changed lines of the file:
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@@
 	)
 	(junction
+		(at 242.57 309.88)
+		(diameter 0)
+		(color 0 0 0 0)
+	)
+	(junction
 		(at 80.01 198.12)
 		(diameter 0)
@@
 	(wire
 		(pts
+			(xy 242.57 309.88) (xy 246.38 309.88)
+		)
+		(stroke
+			(width 0)
+			(type default)
+		)
+	)
+	(wire
+		(pts
 			(xy 152.4 182.88) (xy 152.4 186.69)
 		)
@@
 	(wire
 		(pts
-			(xy 232.41 309.88) (xy 246.38 309.88)
+			(xy 232.41 309.88) (xy 242.57 309.88)
 		)
 		(stroke
@@
 	(wire
 		(pts
+			(xy 242.57 309.88) (xy 242.57 316.23)
+		)
+		(stroke
+			(width 0)
+			(type default)
+		)
+	)
+	(wire
+		(pts
 			(xy 407.67 194.31) (xy 407.67 200.66)
 		)
@@
 	(symbol
 		(lib_id "power:GND")
+		(at 245.11 316.23 90)
+		(unit 1)
+		(exclude_from_sim no)
+		(in_bom yes)
+		(on_board yes)
+		(dnp no)
+		(fields_autoplaced yes)
+		(property "Reference" "#PWR025"
+			(at 251.46 316.23 0)
+			(effects
+				(font
+					(size 1.27 1.27)
+				)
+				(hide yes)
+			)
+		)
+		(property "Value" "AGND"
+			(at 248.92 316.2299 90)
+			(effects
+				(font
+					(size 1.27 1.27)
+				)
+				(justify right)
+			)
+		)
+		(property "Footprint" ""
+			(at 245.11 316.23 0)
+			(effects
+				(font
+					(size 1.27 1.27)
+				)
+				(hide yes)
+			)
+		)
+		(property "Datasheet" ""
+			(at 245.11 316.23 0)
+			(effects
+				(font
+					(size 1.27 1.27)
+				)
+				(hide yes)
+			)
+		)
+		(property "Description" "Power symbol creates a global label with name \"GND\" , ground"
+			(at 245.11 316.23 0)
+			(effects
+				(font
+					(size 1.27 1.27)
+				)
+				(hide yes)
+			)
+		)
+		(pin "1"
+		)
+		(instances
+			(project "Audio_Board_Analog_Only"
+				(path "/5266cf9e-da90-4c53-80fd-cf3dbed42632/e99ff431-6a4b-4cff-9a72-1b9e305d1dd3"
+					(reference "#PWR025")
+					(unit 1)
+				)
+			)
+		)
+	)
+	(symbol
+		(lib_id "power:GND")
 		(at 54.61 138.43 0)
 		(unit 1)
@@
 					(unit 1)
 				)
+			)
+		)
+	)
+	(symbol
+		(lib_id "PCM_SL_Pin_Headers:PINHD_1x2_Male")
+		(at 243.84 320.04 270)
+		(unit 1)
+		(exclude_from_sim no)
+		(in_bom yes)
+		(on_board yes)
+		(dnp no)
+		(fields_autoplaced yes)
+		(property "Reference" "J12"
+			(at 247.65 318.6449 90)
+			(effects
+				(font
+					(size 1.27 1.27)
+				)
+				(justify left)
+			)
+		)
+		(property "Value" "PINHD_1x2_Male"
+			(at 247.65 321.1849 90)
+			(effects
+				(font
+					(size 1.27 1.27)
+				)
+				(justify left)
+			)
+		)
+		(property "Footprint" "Connector_PinHeader_2.54mm:PinHeader_1x02_P2.54mm_Vertical"
+			(at 240.03 321.31 0)
+			(effects
+				(font
+					(size 1.27 1.27)
+				)
+				(hide yes)
+			)
+		)
+		(property "Datasheet" ""
+			(at 251.46 320.04 0)
+			(effects
+				(font
+					(size 1.27 1.27)
+				)
+				(hide yes)
+			)
+		)
+		(property "Description" "Pin Header male with pin space 2.54mm. Pin Count -2"
+			(at 243.84 320.04 0)
+			(effects
+				(font
+					(size 1.27 1.27)
+				)
+				(hide yes)
+			)
+		)
+		(pin "1"
+		)
+		(pin "2"
+		)
+		(instances
+			(project "Audio_Board_Analog_Only"
+				(path "/5266cf9e-da90-4c53-80fd-cf3dbed42632/e99ff431-6a4b-4cff-9a72-1b9e305d1dd3"
+					(reference "J12")
+					(unit 1)
+				)
