File: Audio_Board_Analog_Only/Audio_Board_Analog_Only.kicad_pcb (KiCad board)
At the start: 4 copper layers, 343.1 x 201.9 mm, 261 parts, among them IC1 PCM1865DBT, IC2 LM2940IMPX-10_NOPB, IC3 XC6902NA01PR-G, IC5 PCM1865DBT, J1 Line Out (Left), J10 XLR3_AudioJack3_Combo, J11 PINHD_1x1_Male, J12 PINHD_1x3_Male, J13 PINHD_1x10_Female, J14 PINHD_1x10_Female, J15 PINHD_1x2_Male, J16 PINHD_1x5_Male, J17 PINHD_1x3_Male, J18 PINHD_1x2_Male, J2 Headphone Out, J20 ACJM-MV-2, J21 Line Out (Right), J3 XLR3_AudioJack3_Combo, J4 XLR3_AudioJack3_Combo, J5 ACJM-MV-2, J6 ACJM-MV-2, J7 ACJM-MV-2, J8 PINHD_1x5_Female, J9 XLR3_AudioJack3_Combo, U10 OPA2134, U11 TPA6110A2DGN, U15 OPA2134, U16 SSM2019BRNZ, U17 SSM2019BRNZ, U18 OPA2134, U19 SSM2019BRNZ, U20 SSM2019BRNZ, U34 NE5532AD, U35 NE5532AD, U9 PCM1780

Commit message: made new pcbs :(
Parts:
- removed C222, C223, C226, C227: 10uF, Capacitor_SMD:C_0805_2012Metric
- removed C224, C225: 0.1uF, Capacitor_SMD:C_0603_1608Metric_Pad1.08x0.95mm_HandSolder
- removed C228, C229: 2.2uF, Capacitor_SMD:C_0805_2012Metric
- removed C37: 0.1uF, Capacitor_SMD:C_0805_2012Metric
- removed C38, C39, C40, C43: 10uF, Capacitor_SMD:CP_Elec_4x5.8
- removed C5, C6: 1uF, PCM_Capacitor_SMD_AKL:C_0805_2012Metric
- removed D7: LED, LED_SMD:LED_0402_1005Metric_Pad0.77x0.64mm_HandSolder
- removed IC2: LM2940IMPX-10_NOPB, SamacSys_Parts:SOT230P700X180-4N
- removed J13, J14: PINHD_1x10_Female, Connector_PinSocket_2.54mm:PinSocket_1x10_P2.54mm_Vertical
- removed J15: PINHD_1x2_Male, Connector_PinHeader_2.54mm:PinHeader_1x02_P2.54mm_Vertical
- removed R11, R41: 50, Resistor_SMD:R_0805_2012Metric_Pad1.20x1.40mm_HandSolder
- removed R21: 50, Resistor_SMD:R_0805_2012Metric
- removed R35, R36, R37, R38, R39, R40, R42, R73, R98: 0R, Resistor_SMD:R_0805_2012Metric_Pad1.20x1.40mm_HandSolder
- removed R43, R72: 2.2k, Resistor_SMD:R_0805_2012Metric_Pad1.20x1.40mm_HandSolder
- removed R90, R91, R92, R93, R94, R95, R96, R97: 100k, PCM_Resistor_SMD_AKL:R_0402_1005Metric
- removed U9: PCM1780, Package_SO:SSOP-16_3.9x4.9mm_P0.635mm
- added C10: 1uF, PCM_Capacitor_SMD_AKL:C_0805_2012Metric, F.Cu at (317.7, 161.9)
- added C11: 1uF, PCM_Capacitor_SMD_AKL:C_0805_2012Metric, F.Cu at (311.8, 165.8)
- added C12: 0.47uF, PCM_Capacitor_SMD_AKL:C_0805_2012Metric, F.Cu at (182.9, 97.6)
- added C13: 22uF, Capacitor_SMD:CP_Elec_4x5.8, F.Cu at (182.9, 108.9)
- added C18: 1uF, PCM_Capacitor_SMD_AKL:C_0805_2012Metric, F.Cu at (251.0, 115.6)
- added C23: 1uF, PCM_Capacitor_SMD_AKL:C_0805_2012Metric, F.Cu at (330.1, 143.9)
- added C24: 1uF, Capacitor_SMD:C_0402_1005Metric, F.Cu at (327.3, 113.0)
- added C25: 1uF, Capacitor_SMD:C_0402_1005Metric, F.Cu at (326.2, 110.2)
- added D10: LED, LED_SMD:LED_0402_1005Metric_Pad0.77x0.64mm_HandSolder, F.Cu at (327.9, 127.1)
- added D11: LED, LED_SMD:LED_0402_1005Metric_Pad0.77x0.64mm_HandSolder, F.Cu at (333.1, 149.5)
- added D9: LED, LED_SMD:LED_0402_1005Metric_Pad0.77x0.64mm_HandSolder, F.Cu at (246.6, 110.7)
- added IC10: XC6902NA01PR-G, SamacSys_Parts:XC6902NA01PRG, F.Cu at (334.8, 143.3)
- added IC4: XC6902NA01PR-G, SamacSys_Parts:XC6902NA01PRG, F.Cu at (316.6, 166.4)
- added IC6: XC6902NA01PR-G, SamacSys_Parts:XC6902NA01PRG, F.Cu at (186.5, 88.2)
- added IC7: LM2940IMPX-10_NOPB, SamacSys_Parts:SOT230P700X180-4N, F.Cu at (272.4, 111.8)
- added IC8: XC6902NA01PR-G, SamacSys_Parts:XC6902NA01PRG, F.Cu at (252.1, 111.1)
- added IC9: LM2940IMPX-10_NOPB, SamacSys_Parts:SOT230P700X180-4N, F.Cu at (337.8, 130.1)
- C1: value 10uF -> 1uF; footprint Capacitor_SMD:C_0805_2012Metric -> Capacitor_SMD:C_0402_1005Metric
- C14, C15, C19: value 10uF -> 1uF; footprint Capacitor_SMD:C_0805_2012Metric -> PCM_Capacitor_SMD_AKL:C_0805_2012Metric
- C16: value 0.1uF -> 0.47uF; footprint Capacitor_SMD:C_0603_1608Metric_Pad1.08x0.95mm_HandSolder -> PCM_Capacitor_SMD_AKL:C_0805_2012Metric
- C17: value 0.1uF -> 22uF; footprint Capacitor_SMD:C_0603_1608Metric_Pad1.08x0.95mm_HandSolder -> Capacitor_SMD:CP_Elec_4x5.8
- C2: value 10uF -> 0.1uF; footprint Capacitor_SMD:C_0805_2012Metric -> Capacitor_SMD:C_0402_1005Metric
- C20, C3: value 10uF -> 0.47uF; footprint Capacitor_SMD:C_0805_2012Metric -> PCM_Capacitor_SMD_AKL:C_0805_2012Metric
- C21: value 2.2uF -> 22uF; footprint Capacitor_SMD:C_0805_2012Metric -> Capacitor_SMD:CP_Elec_4x5.8
- C22: value 2.2uF -> 1uF; footprint Capacitor_SMD:C_0805_2012Metric -> PCM_Capacitor_SMD_AKL:C_0805_2012Metric
- C4: value 10uF -> 22uF; footprint Capacitor_SMD:C_0805_2012Metric -> Capacitor_SMD:CP_Elec_4x5.8
- C7: value 0.47uF -> 0.01uF; footprint PCM_Capacitor_SMD_AKL:C_0805_2012Metric -> Capacitor_SMD:C_0402_1005Metric
- C8: value 22uF -> 0.001uF; footprint Capacitor_SMD:CP_Elec_4x5.8 -> Capacitor_SMD:C_0402_1005Metric
- IC1, IC5: value PCM1865DBT -> LM2940IMPX-10_NOPB; footprint SamacSys_Parts:SOP50P640X120-30N -> SamacSys_Parts:SOT230P700X180-4N
- IC3: value XC6902NA01PR-G -> TPS73250DBVR; footprint SamacSys_Parts:XC6902NA01PRG -> SamacSys_Parts:SOT95P280X145-5N
- J11: value PINHD_1x1_Male -> SBH11-PBPC-D10-ST-BK; footprint Connector_PinHeader_2.54mm:PinHeader_1x01_P2.54mm_Vertical -> SamacSys_Parts:SHDR20W64P254_2X10_2794X910X880P
- J12: value PINHD_1x3_Male -> PINHD_1x2_Male; footprint Connector_PinHeader_2.54mm:PinHeader_1x03_P2.54mm_Vertical -> Connector_PinHeader_2.54mm:PinHeader_1x02_P2.54mm_Vertical
- R1, R2: value 0R -> 0; footprint Resistor_SMD:R_0805_2012Metric_Pad1.20x1.40mm_HandSolder -> Resistor_SMD:R_0805_2012Metric
- R12: value 50 -> 0; footprint Resistor_SMD:R_0805_2012Metric_Pad1.20x1.40mm_HandSolder -> Resistor_SMD:R_0805_2012Metric
- R13, R15, R16: value 2.2k -> 0
- R19, R22: value 50 -> 0
- R20: value 0R -> 0
- R3, R34, R8: value 0R -> 2.2k; footprint Resistor_SMD:R_0805_2012Metric_Pad1.20x1.40mm_HandSolder -> Resistor_SMD:R_0805_2012Metric
- R4: value 0 -> 2.2k; footprint Resistor_SMD:R_0805_2012Metric_Pad1.20x1.40mm_HandSolder -> Resistor_SMD:R_0805_2012Metric
- R9: value 50 -> 2.2k; footprint Resistor_SMD:R_0805_2012Metric_Pad1.20x1.40mm_HandSolder -> Resistor_SMD:R_0805_2012Metric
- moved R3 239.2 mm to (346.6, 156.9)
- moved R10 221.3 mm to (335.7, 150.1), turned to 0 degrees
- moved C20 217.7 mm to (343.0, 125.2), turned to 90 degrees
- moved C22 214.7 mm to (339.2, 144.4), turned to -90 degrees
- moved C21 210.2 mm to (331.3, 128.4)
- moved R34 204.5 mm to (321.6, 107.6), turned to 180 degrees
- moved IC1 202.3 mm to (335.1, 158.9), turned to 90 degrees
- moved C1 187.8 mm to (323.4, 119.0), turned to 180 degrees
- moved D2 184.8 mm to (308.8, 167.3), turned to -90 degrees
- moved C2 181.7 mm to (323.4, 117.7), turned to 180 degrees
- moved R4 179.5 mm to (308.8, 170.4), turned to -90 degrees
- moved R1 178.3 mm to (333.7, 167.5), turned to 0 degrees
- moved R9 173.6 mm to (326.2, 129.3), turned to -90 degrees
- moved D1 164.3 mm to (346.6, 160.1)
- moved C16 155.3 mm to (277.2, 107.5), turned to 90 degrees
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Connections:
- C1 pad 1: Net-(IC1-VINL2/VIN1M) -> AGND
- C1 pad 2: AIN_3 -> Net-(IC3-EN)
- C106 pad 1: -12V -> -12V_Preamp1
- C107 pad 1: -12V -> -12V_Preamp1
- C108 pad 1: 12V -> 12V_Preamp1
- C109 pad 1: 12V -> 12V_Preamp1
- C14 pad 1: AGND -> Net-(IC6--VIN)
- C14 pad 2: Net-(IC1-AVDD) -> AGND
- C15 pad 1: 3.3V_2 -> -12V_Preamp1
- C15 pad 2: DGND -> AGND
- C16 pad 1: AGND -> Net-(IC7-IN)
- C16 pad 2: Net-(IC1-AVDD) -> AGND
- C17 pad 1: 3.3V_2 -> 12V_Preamp2
- C17 pad 2: DGND -> AGND
- C19 pad 1: AIN_2 -> -12V_Preamp2
- C19 pad 2: Net-(IC1-VINR1/VIN2P) -> AGND
- C2 pad 1: Net-(IC1-VINR2/VIN2M) -> AGND
- C2 pad 2: AIN_4 -> Net-(IC3-EN)
- C20 pad 1: AIN_1 -> Net-(IC9-IN)
- C20 pad 2: Net-(IC1-VINL1/VIN1P) -> AGND
- C21 pad 1: AGND -> 12V_Outputs
- C21 pad 2: Net-(IC1-VREF) -> AGND
- C22 pad 1: DGND -> Net-(IC10--VIN)
- C22 pad 2: Net-(IC1-LDO) -> AGND
- C3 pad 1: Net-(IC5-VINL2/VIN1M) -> Net-(IC1-IN)
- C3 pad 2: AIN_7 -> AGND
- C4 pad 1: Net-(IC5-VINR2/VIN2M) -> 12V_Filtered
- C4 pad 2: AIN_8 -> AGND
- C41 pad 1: 12V -> 12V_Outputs
- C42 pad 2: -12V -> -12V_Outputs
- C46 pad 1: 5V -> 5V_Filtered
- C7 pad 1: REAL_12V -> AGND
- C7 pad 2: AGND -> Net-(IC3-EN)
- C76 pad 2: 12V -> 12V_Preamp2
- C77 pad 2: -12V -> -12V_Preamp2
- C78 pad 1: -12V -> -12V_Preamp1
- C79 pad 1: -12V -> -12V_Preamp1
- C8 pad 1: 12V -> AGND
- C8 pad 2: AGND -> Net-(IC3-EN)
- C82 pad 1: 12V -> 12V_Preamp1
- C83 pad 1: 12V -> 12V_Preamp1
- C84 pad 2: 12V -> 12V_Preamp2
- C85 pad 2: -12V -> -12V_Preamp2
- C9 pad 1: 5V -> 5V_Filtered
- D1 pad 2: Net-(IC5-AVDD) -> 12V_Filtered
- D2 pad 1: Net-(D2-Pad1) -> -12V_Filtered
- D2 pad 2: 3.3V_2 -> Net-(D2-Pad2)
- D3 pad 2: 3.3V_2 -> 12V_Preamp1
- D4 pad 1: Net-(D4-Pad1) -> -12V_Preamp1
- D4 pad 2: Net-(IC1-AVDD) -> Net-(D4-Pad2)
- D5 pad 2: 5V -> 12V_Preamp2
- D6 pad 2: 5V -> 5V_Filtered
- D8 pad 2: 12V -> 5V_Filtered
- IC1 pad 1: Net-(IC1-VINL2/VIN1M) -> Net-(IC1-IN)
- IC1 pad 2: Net-(IC1-VINR2/VIN2M) -> AGND
- IC1 pad 3: Net-(IC1-VINL1/VIN1P) -> 12V_Filtered
- IC1 pad 4: Net-(IC1-VINR1/VIN2P) -> AGND
- IC3 pad 1: AGND -> Net-(IC3-EN)
- IC3 pad 2: REAL_-12V -> AGND
- IC3 pad 3: -12V -> Net-(IC3-EN)
- IC3 pad 4: REAL_-12V -> Net-(IC3-NR/FB)
- IC5 pad 1: Net-(IC5-VINL2/VIN1M) -> Net-(IC5-IN)
- IC5 pad 2: Net-(IC5-VINR2/VIN2M) -> AGND
- IC5 pad 3: Net-(IC5-VINL1/VIN1P) -> 12V_Preamp1
- IC5 pad 4: Net-(IC5-VINR1/VIN2P) -> AGND
- J11 pad 1: 3.3V_2 -> AIN_1
- J12 pad 1: Net-(U9-~{MS}) -> AGND
- J12 pad 2: Net-(U9-MC) -> AIN_8
- J16 pad 2: 5V -> AGND
- J16 pad 3: REAL_-12V -> 5V
- J16 pad 4: REAL_12V -> REAL_-12V
- J16 pad 5: 3.3V -> REAL_12V
- J8 pad 1: 3.3V -> REAL_12V
- J8 pad 2: REAL_12V -> REAL_-12V
- J8 pad 3: REAL_-12V -> 5V
- J8 pad 4: 5V -> AGND
- R1 pad 1: DGND -> Net-(IC1-IN)
- R1 pad 2: AGND -> REAL_12V
- R10 pad 1: Net-(D4-Pad1) -> Net-(D11-Pad2)
- R12 pad 1: DIN -> Net-(IC5-IN)
- R12 pad 2: Net-(J13-Pad2) -> 12V_Filtered
- R13 pad 1: Net-(D5-Pad1) -> Net-(IC6--VIN)
- R13 pad 2: AGND -> -12V_Filtered
- R15 pad 2: AGND -> -12V_Filtered
- R16 pad 1: Net-(D8-Pad1) -> Net-(IC7-IN)
- R16 pad 2: AGND -> 12V_Filtered
- R19 pad 1: BCLK_DAC -> Net-(IC9-IN)
- R19 pad 2: Net-(U9-BCK) -> 12V_Filtered
- R2 pad 1: DGND -> Net-(IC4--VIN)
- R2 pad 2: AGND -> REAL_-12V
- R20 pad 1: MCLK -> Net-(IC10--VIN)
- R20 pad 2: Net-(U9-SCK) -> -12V_Filtered
- R22 pad 1: DATA -> Net-(IC3-EN)
- R22 pad 2: Net-(U9-DATA) -> 5V
- R27 pad 1: Net-(C34-Pad2) -> LEFT_IN
- R27 pad 2: LEFT_IN -> Net-(C34-Pad2)
- R3 pad 1: DGND -> Net-(D1-Pad1)
- R34 pad 1: 3.3V -> Net-(D8-Pad1)
- R34 pad 2: Net-(IC1-AVDD) -> AGND
- R4 pad 1: MCLK -> Net-(D2-Pad2)
- R4 pad 2: Net-(IC1-SCKI) -> AGND
- R5 pad 2: DGND -> AGND
- R6 pad 1: Net-(D1-Pad1) -> Net-(D4-Pad2)
- R7 pad 1: Net-(D2-Pad1) -> Net-(D5-Pad1)
- R7 pad 2: DGND -> AGND
- R8 pad 1: LRCK_DAC -> Net-(D9-Pad2)
- R8 pad 2: Net-(J13-Pad7) -> AGND
- R9 pad 1: BCLK_ADC -> Net-(D10-Pad1)
- R9 pad 2: Net-(J13-Pad4) -> AGND
- U10 pad 4: -12V -> -12V_Outputs
- U10 pad 8: 12V -> 12V_Outputs
- U11 pad 6: 5V -> 5V_Filtered
- U15 pad 4: -12V -> -12V_Preamp2
- U15 pad 8: 12V -> 12V_Preamp2
- U16 pad 4: -12V -> -12V_Preamp1
- U16 pad 7: 12V -> 12V_Preamp1
- U17 pad 4: -12V -> -12V_Preamp1
- U17 pad 7: 12V -> 12V_Preamp1
- U18 pad 4: -12V -> -12V_Preamp2
- U18 pad 8: 12V -> 12V_Preamp2
- U19 pad 4: -12V -> -12V_Preamp1
- U19 pad 7: 12V -> 12V_Preamp1
- U20 pad 4: -12V -> -12V_Preamp1
- U20 pad 7: 12V -> 12V_Preamp1
- U34 pad 4: -12V -> -12V_Outputs
- U34 pad 8: 12V -> 12V_Outputs
- U35 pad 4: -12V -> -12V_Outputs
- U35 pad 8: 12V -> 12V_Outputs
Routing:
- net 12V: track 549.0 -> 0.00 mm, vias 11 -> 0
- net -12V: track 535.7 -> 0.00 mm, vias 14 -> 0
- net 3.3V: track 273.3 -> 0.00 mm, vias 5 -> 0
- net MCLK: track 260.7 -> 0.00 mm, vias 4 -> 0
- net 12V_Filtered: track 0.00 -> 255.7 mm, vias 0 -> 4
- net -12V_Preamp1: track 0.00 -> 244.8 mm, vias 0 -> 6
- net 3.3V_2: track 227.3 -> 0.00 mm, vias 2 -> 0
- net -12V_Filtered: track 0.00 -> 217.1 mm, vias 0 -> 5
- net 12V_Preamp1: track 0.00 -> 195.1 mm, vias 0 -> 4
- net LRCK_DAC: track 155.0 -> 0.00 mm, vias 2 -> 0
- net BCLK_DAC: track 148.3 -> 0.00 mm, vias 2 -> 0
- net SDA: track 146.0 -> 0.00 mm, vias 6 -> 0
- net DATA: track 143.7 -> 0.00 mm, vias 2 -> 0
- net SCL: track 140.7 -> 0.00 mm, vias 6 -> 0
- net -12V_Outputs: track 0.00 -> 137.6 mm, vias 0 -> 3
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- added copper zone on In2.Cu, net AGND
- removed copper zone on F.Cu, net DGND
- removed copper zone on In2.Cu, net DGND
Other:
- board size 343.1 x 201.9 mm -> 336.7 x 152.9 mm
- board text added: "Analog Board"
- board text added: "V1"
- board text removed: "3.3V"
- board text removed: "3.3V (Digital)"
- board text removed: "Audio Board"
- board text removed: "DAC"
- board text removed: "DGND"
- board text removed: "Left ADC"
- board text removed: "Pins to MCU"
- board text removed: "Right ADC"
- board text removed: "V2 :("

Commit message: aaaah (cooked)
Other:
- board size 336.7 x 152.9 mm -> 327.8 x 144.6 mm
