File: Audio_Board_AD_Breakout/Audio_Board_AD_Breakout.kicad_pcb (KiCad board)
At the start: 4 copper layers, 343.1 x 201.9 mm, 261 parts, among them IC1 PCM1865DBT, IC2 LM2940IMPX-10_NOPB, IC3 XC6902NA01PR-G, IC5 PCM1865DBT, J1 Line Out (Left), J10 XLR3_AudioJack3_Combo, J11 PINHD_1x1_Male, J12 PINHD_1x3_Male, J13 PINHD_1x10_Female, J14 PINHD_1x10_Female, J15 PINHD_1x2_Male, J16 PINHD_1x5_Male, J17 PINHD_1x3_Male, J18 PINHD_1x2_Male, J2 Headphone Out, J20 ACJM-MV-2, J21 Line Out (Right), J3 XLR3_AudioJack3_Combo, J4 XLR3_AudioJack3_Combo, J5 ACJM-MV-2, J6 ACJM-MV-2, J7 ACJM-MV-2, J8 PINHD_1x5_Female, J9 XLR3_AudioJack3_Combo, U10 OPA2134, U11 TPA6110A2DGN, U15 OPA2134, U16 SSM2019BRNZ, U17 SSM2019BRNZ, U18 OPA2134, U19 SSM2019BRNZ, U20 SSM2019BRNZ, U34 NE5532AD, U35 NE5532AD, U9 PCM1780

Commit message: made new pcbs :(
Parts:
- removed C100, C101, C102, C103, C70, C71, C72, C73: 47 uF, Capacitor_SMD:CP_Elec_4x5.8
- removed C104, C105, C54, C55, C62, C63, C74, C75, C86, C87, C92, C93: 200pF, Capacitor_SMD:C_0603_1608Metric_Pad1.08x0.95mm_HandSolder
- removed C106, C107, C108, C109, C58, C59, C76, C77, C78, C79, C80, C81, C82, C83, C84, C85: 0.1uF, Capacitor_SMD:C_0603_1608Metric_Pad1.08x0.95mm_HandSolder
- removed C29, C30: 1200pF, Capacitor_SMD:C_0603_1608Metric_Pad1.08x0.95mm_HandSolder
- removed C34, C36: 120pF, Capacitor_SMD:C_0603_1608Metric_Pad1.08x0.95mm_HandSolder
- removed C41, C42: 10uF, Capacitor_SMD:CP_Elec_4x5.8
- removed C44, C45, C46, C48: 1uF, Capacitor_SMD:C_0805_2012Metric
- removed C56, C57, C60, C61, C88, C89, C90, C91: 470pF, Capacitor_SMD:C_0603_1608Metric_Pad1.08x0.95mm_HandSolder
- removed C64, C67, C94, C97: 47uF, Capacitor_SMD:CP_Elec_4x5.8
- removed C65, C66, C68, C69, C95, C96, C98, C99: 22uF, Capacitor_SMD:C_0603_1608Metric_Pad1.08x0.95mm_HandSolder
- removed D6, D7, D8: LED, LED_SMD:LED_0402_1005Metric_Pad0.77x0.64mm_HandSolder
- removed DZ1, DZ10, DZ11, DZ12, DZ13, DZ14, DZ15, DZ16, DZ2, DZ3, DZ4, DZ5, DZ6, DZ7, DZ8, DZ9: 10V, Diode_SMD:D_SMB
- removed IC2: LM2940IMPX-10_NOPB, SamacSys_Parts:SOT230P700X180-4N
- removed J10, J3, J4, J9: XLR3_AudioJack3_Combo, Connector_Audio:Jack_XLR-6.35mm_Neutrik_NCJ6FA-V_Vertical
- removed J16: PINHD_1x5_Male, Connector_PinHeader_2.54mm:PinHeader_1x05_P2.54mm_Vertical
- removed J17: PINHD_1x3_Male, Connector_PinHeader_2.54mm:PinHeader_1x03_P2.54mm_Vertical
- removed J18: PINHD_1x2_Male, Connector_PinHeader_2.54mm:PinHeader_1x02_P2.54mm_Vertical
- removed J2: Headphone Out, SamacSys_Parts:ACJSNV353
- removed J20, J5, J6, J7: ACJM-MV-2, SamacSys_Parts:ACJMMV2
- removed J21: Line Out (Right), SamacSys_Parts:ACJSNV353
- removed R16, R58, R59, R60, R61, R62, R63, R70, R71, R84, R85, R86, R87: 2.2k, Resistor_SMD:R_0805_2012Metric
- removed R167, R168, R169, R170: 3k, Resistor_SMD:R_0805_2012Metric
- removed R17, R18: 8.2k, Resistor_SMD:R_0805_2012Metric
- removed R23, R24, R55, R57, R68, R69: 1k, Resistor_SMD:R_0805_2012Metric
- removed R25, R26: 15k, Resistor_SMD:R_0805_2012Metric
- removed R27, R28: 100, Resistor_SMD:R_0805_2012Metric
- removed R29, R30: 20k, Resistor_SMD:R_0805_2012Metric
- removed R31, R32, R33: 82k, Resistor_SMD:R_0805_2012Metric
- removed R44, R45, R46, R47, R74, R75, R76, R77: 5.1k, Resistor_SMD:R_0805_2012Metric
- removed R48, R49, R66, R67: 1M, Resistor_SMD:R_0805_2012Metric
- removed R50, R51, R52, R53, R78, R79, R80, R81: 10k, Resistor_SMD:R_0805_2012Metric
- removed R54, R56, R82, R83: 47, Resistor_SMD:R_0805_2012Metric
- removed R64, R65, R88, R89: 1.1k, Resistor_SMD:R_0805_2012Metric
- removed U10, U15, U18: OPA2134, SamacSys_Parts:SOIC127P600X175-8N
- removed U11: TPA6110A2DGN, Package_SO:HVSSOP-8-1EP_3x3mm_P0.65mm_EP1.57x1.89mm
- removed U16, U17, U19, U20: SSM2019BRNZ, SamacSys_Parts:SOIC127P600X175-8N
- removed U34, U35: NE5532AD, PCM_Package_SO_AKL:SO-8_3.9x4.9mm_P1.27mm
- added C10: 1uF, Capacitor_SMD:C_0402_1005Metric, F.Cu at (266.1, 143.0)
- added C11: 0.1uF, Capacitor_SMD:C_0402_1005Metric, F.Cu at (266.1, 144.3)
- added C12: 0.01uF, Capacitor_SMD:C_0402_1005Metric, F.Cu at (266.1, 145.6)
- added C13: 0.001uF, Capacitor_SMD:C_0402_1005Metric, F.Cu at (266.1, 146.8)
- added C18: 1uF, Capacitor_SMD:C_0402_1005Metric, F.Cu at (264.2, 136.9)
- added C23: 1uF, Capacitor_SMD:C_0402_1005Metric, F.Cu at (266.0, 140.9)
- added C24: 1uF, Capacitor_SMD:C_0402_1005Metric, F.Cu at (254.2, 142.9)
- added IC4: TPS73250DBVR, SamacSys_Parts:SOT95P280X145-5N, F.Cu at (253.4, 139.9)
- C5, C6: footprint PCM_Capacitor_SMD_AKL:C_0805_2012Metric -> Capacitor_SMD:C_0402_1005Metric
- C7: value 0.47uF -> 0.1uF; footprint PCM_Capacitor_SMD_AKL:C_0805_2012Metric -> Capacitor_SMD:C_0402_1005Metric
- C8: value 22uF -> 0.01uF; footprint Capacitor_SMD:CP_Elec_4x5.8 -> Capacitor_SMD:C_0402_1005Metric
- C9: value 10uF -> 0.001uF; footprint Capacitor_SMD:CP_Elec_4x5.8 -> Capacitor_SMD:C_0402_1005Metric
- IC3: value XC6902NA01PR-G -> TPS73250DBVR; footprint SamacSys_Parts:XC6902NA01PRG -> SamacSys_Parts:SOT95P280X145-5N
- J1: value Line Out (Left) -> SBH11-PBPC-D10-ST-BK; footprint SamacSys_Parts:ACJSNV353 -> SamacSys_Parts:SHDR20W64P254_2X10_2794X910X880P
- R14, R15: value 2.2k -> 0
- moved H1 247.5 mm to (268.7, 119.0)
- moved H2 245.2 mm to (107.2, 119.0)
- moved J1 143.5 mm to (154.1, 132.4)
- moved R15 109.5 mm to (255.4, 146.1)
- moved C6 109.3 mm to (255.1, 136.8), turned to 0 degrees
- moved R13 109.0 mm to (223.8, 117.7), turned to 180 degrees
- moved C5 105.7 mm to (249.6, 147.0), turned to 0 degrees
- moved D5 105.6 mm to (227.1, 119.3), turned to 0 degrees
- moved R21 103.8 mm to (246.3, 117.8), turned to 180 degrees
- moved C37 102.7 mm to (232.1, 120.2), turned to 90 degrees
- moved C43 101.9 mm to (224.6, 122.8), turned to 180 degrees
- moved C38 100.9 mm to (236.4, 120.7), turned to 90 degrees
- moved R19 100.0 mm to (246.3, 120.5), turned to 180 degrees
- moved C9 99.7 mm to (249.6, 143.0)
- moved C8 97.2 mm to (249.6, 145.6), turned to 0 degrees
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Connections:
- C37 pad 1: 5V -> 5V_Filtered
- C38 pad 1: 5V -> 5V_Filtered
- C5 pad 1: REAL_-12V -> AGND
- C5 pad 2: AGND -> Net-(IC4-EN)
- C6 pad 1: -12V -> 3.3V_Filtered
- C7 pad 1: REAL_12V -> AGND
- C7 pad 2: AGND -> Net-(IC4-EN)
- C8 pad 1: 12V -> AGND
- C8 pad 2: AGND -> Net-(IC4-EN)
- C9 pad 1: 5V -> AGND
- C9 pad 2: AGND -> Net-(IC4-EN)
- D5 pad 2: 5V -> 5V_Filtered
- IC3 pad 1: AGND -> Net-(IC3-EN)
- IC3 pad 2: REAL_-12V -> AGND
- IC3 pad 3: -12V -> Net-(IC3-EN)
- IC3 pad 4: REAL_-12V -> Net-(IC3-NR/FB)
- J1 pad 1: AGND -> AIN_1
- J1 pad 3: LEFT_OUT- -> AIN_2
- J1 pad 4: LEFT_OUT+ -> AGND
- J8 pad 2: REAL_12V -> unconnected-(J8-Pad2)
- J8 pad 3: REAL_-12V -> 5V
- J8 pad 4: 5V -> unconnected-(J8-Pad4)
- R14 pad 1: Net-(D6-Pad1) -> Net-(IC3-EN)
- R14 pad 2: AGND -> 5V
- R15 pad 1: Net-(D7-Pad2) -> Net-(IC4-EN)
- R15 pad 2: AGND -> 3.3V
- R34 pad 1: 3.3V -> 3.3V_Filtered
- R73 pad 1: 3.3V -> 3.3V_Filtered
- R98 pad 2: 3.3V -> 3.3V_2
- U9 pad 11: 5V -> 5V_Filtered
Routing:
- net 12V: track 549.0 -> 0.00 mm, vias 11 -> 0
- net -12V: track 535.7 -> 0.00 mm, vias 14 -> 0
- net 3.3V: track 273.3 -> 3.79 mm, vias 5 -> 0
- net AGND: track 332.7 -> 102.8 mm, vias 135 -> 56
- net 5V: track 204.5 -> 3.74 mm, vias 4 -> 0
- net 36V: track 186.3 -> 0.00 mm, vias 6 -> 0
- net 3.3V_Filtered: track 0.00 -> 157.6 mm, vias 0 -> 3
- net 3.3V_2: track 227.3 -> 361.0 mm
- net Net-(C102-Pad1): track 108.2 -> 0.00 mm, vias 5 -> 0
- net Net-(C63-Pad2): track 95.4 -> 0.00 mm, vias 5 -> 0
- net LEFT_IN: track 88.8 -> 0.00 mm, vias 2 -> 0
- net Net-(C100-Pad1): track 88.7 -> 0.00 mm, vias 5 -> 0
- net RIGHT_IN: track 82.7 -> 0.00 mm, vias 2 -> 0
- net LEFT_OUT+: track 81.4 -> 0.00 mm, vias 2 -> 0
- net Net-(C62-Pad2): track 81.3 -> 0.00 mm, vias 5 -> 0
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- removed copper zone on F.Cu, net (none)
Other:
- board size 343.1 x 201.9 mm -> 171.5 x 103.6 mm
- board text added: "3.3V (A)"
- board text added: "3.3V (D)"
- board text added: "Mister Mixer ADC/DAC Board V1"
- board text added: "Pins to Main Board"
- board text removed: "-12V"
- board text removed: "12V"
- board text removed: "3.3V"
- board text removed: "30mm Apart"
- board text removed: "36V"
- board text removed: "Audio Board"
- board text removed: "Headphone Amplifier"
- board text removed: "Headphone Out"
- board text removed: "L"
- board text removed: "Left Out (+/-)"
- board text removed: "Line Out"
- board text removed: "MISTER MIXER"
- board text removed: "Post-DAC LPF"
- board text removed: "R"
- board text removed: "Right Out (+/-)"
- board text removed: "Test Point"
- board text removed: "V2 :("

Commit message: aaaah (cooked)
Parts:
- added C25: 1uF, Capacitor_SMD:C_0402_1005Metric, F.Cu at (115.4, 199.2)
- added C26: 0.1uF, Capacitor_SMD:C_0402_1005Metric, F.Cu at (115.5, 200.3)
- added C27: 0.01uF, Capacitor_SMD:C_0402_1005Metric, F.Cu at (115.5, 201.6)
- added C28: 0.001uF, Capacitor_SMD:C_0402_1005Metric, F.Cu at (115.5, 202.8)
- added C29: 1uF, Capacitor_SMD:C_0402_1005Metric, F.Cu at (118.5, 210.8)
- added C30: 1uF, Capacitor_SMD:C_0402_1005Metric, F.Cu at (118.0, 205.6)
- added IC2: TPS73250DBVR, SamacSys_Parts:SOT95P280X145-5N, F.Cu at (116.8, 208.3)
- added R16: 0, Resistor_SMD:R_0805_2012Metric, F.Cu at (111.3, 199.2)
Connections:
- J11 pad 1: 3.3V_2 -> 3.3V_Digital
Routing:
- net Net-(IC2-EN): track 0.00 -> 18.9 mm
- net 3.3V_2: track 361.0 -> 349.1 mm
- net DGND: track 33.3 -> 42.9 mm, vias 17 -> 24
- net 3.3V_Digital: track 0.00 -> 3.19 mm
- net Net-(IC2-NR/FB): track 0.00 -> 1.61 mm
