File: Audio_Board_AD_Breakout/Phantom.kicad_sch (KiCad schematic)
At the start: 30 parts, among them IC2 TLV73333PDBVR, IC3 LM2940IMPX-10_NOPB, J1 PINHD_1x10_Male, J11 PINHD_1x1_Male, J13 PINHD_1x10_Female, J14 PINHD_1x10_Female, J16 PINHD_1x5_Male, J3 PINHD_1x10_Male, J8 PINHD_1x5_Female

Commit message: made new pcbs :(
Parts:
- removed C10: 0.47uF, PCM_Capacitor_SMD_AKL:C_0805_2012Metric, symbol PCM_Capacitor_AKL:C_0805
- removed C11: 22uF, Capacitor_SMD:CP_Elec_4x5.8, symbol Device:C_Polarized_US
- removed D6: LED, LED_SMD:LED_0402_1005Metric_Pad0.77x0.64mm_HandSolder, symbol PCM_SL_Devices:LED
- removed IC2: TLV73333PDBVR, symbol SamacSys_Parts:TLV73333PDBVR
- removed IC3: LM2940IMPX-10_NOPB, SamacSys_Parts:SOT230P700X180-4N, symbol SamacSys_Parts:LM2940IMPX-10_NOPB
- removed J1, J3: PINHD_1x10_Male, Connector_Header_2.54mm:PinHeader_1x10_P2.54mm_Vertical, symbol PCM_SL_Pin_Headers:PINHD_1x10_Female
- removed J16: PINHD_1x5_Male, Connector_PinHeader_2.54mm:PinHeader_1x05_P2.54mm_Vertical, symbol PCM_SL_Pin_Headers:PINHD_1x5_Male
- removed R16: 0, Resistor_SMD:R_0805_2012Metric, symbol Device:R
- added C10, C18, C23, C24: 1uF, Capacitor_SMD:C_0402_1005Metric, symbol Device:C
- added C11: 0.1uF, Capacitor_SMD:C_0402_1005Metric, symbol Device:C
- added C12: 0.01uF, Capacitor_SMD:C_0402_1005Metric, symbol Device:C
- added C13: 0.001uF, Capacitor_SMD:C_0402_1005Metric, symbol Device:C
- added H1, H2, H3, H4: MountingHole_M3, MountingHole:MountingHole_3.2mm_M3, symbol PCM_SL_Mechanical:MountingHole_M3
- added IC3, IC4: TPS73250DBVR, SOT95P280X145-5N, symbol SamacSys_Parts:TPS73250DBVR
- added J1: SBH11-PBPC-D10-ST-BK, SHDR20W64P254_2X10_2794X910X880P, symbol SamacSys_Parts:SBH11-PBPC-D10-ST-BK
- R14: value 2.2k -> 0
Connections:
- net 3.3V_2: no longer J8.2
- net 3.3V_Filtered: now also IC4.5 (OUT)
- net 5V: now also R14.2
- net 5V_Filtered: now also C18.1, IC3.5 (OUT)
- net AGND: now also C10.1, C11.1, C12.1, C13.1, C18.2, C23.1, C24.1, IC3.2 (GND), IC4.2 (GND), J1.10, J1.12, J1.14, J1.16, J1.18, J1.2, J1.20, J1.4, J1.6, J1.8; no longer R14.2
- net AIN_1: now also J1.1
- net AIN_2: now also J1.3
- net AIN_3: now also J1.5
- net AIN_4: now also J1.7
- net AIN_5: now also J1.9
- net AIN_6: now also J1.11
- net AIN_7: now also J1.13
- net AIN_8: now also J1.15
- net VOUT_L: now also J1.17
- net VOUT_R: now also J1.19
- net at C5.2, C7.2, C8.2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: now also IC4.1 (IN), IC4.3 (EN)
- net at R14.1: now also C10.2, C11.2, C12.2, C13.2, IC3.1 (IN), IC3.3 (EN)
- new net: C24.2, IC4.4 (NR/FB)
- new net: C23.2, IC3.4 (NR/FB)
Other:
- moved on the sheet: C6

Commit message: aaaah (cooked)
Parts:
- added C25, C29, C30: 1uF, Capacitor_SMD:C_0402_1005Metric, symbol Device:C
- added C26: 0.1uF, Capacitor_SMD:C_0402_1005Metric, symbol Device:C
- added C27: 0.01uF, Capacitor_SMD:C_0402_1005Metric, symbol Device:C
- added C28: 0.001uF, Capacitor_SMD:C_0402_1005Metric, symbol Device:C
- added IC2: TPS73250DBVR, SOT95P280X145-5N, symbol SamacSys_Parts:TPS73250DBVR
- added R16: 0, Resistor_SMD:R_0805_2012Metric, symbol Device:R
Connections:
- net 3.3V_2: now also C30.1, IC2.5 (OUT); no longer J11.1
- net DGND: now also C25.1, C26.1, C27.1, C28.1, C29.1, C30.2, IC2.2 (GND)
- new net: C25.2, C26.2, C27.2, C28.2, IC2.1 (IN), IC2.3 (EN), R16.1
- new net: C29.2, IC2.4 (NR/FB)
- new net 3.3V_Digital: J11.1, R16.2
Other:
- moved on the sheet: J11
